File: schem/LED_driver/LED_driver.sch (KiCad schematic (older format))
At the start: 137 parts

Commit message: Закончена схема
Parts:
- removed C? (x25): 0.1mkF, Capacitor_SMD:C_0805_2012Metric, symbol Device:C
- removed C? (x10): 470mkF, Capacitor_THT:CP_Radial_D10.0mm_P5.00mm, symbol Device:CP
- removed C? (x5): 1mkF, Capacitor_SMD:C_0805_2012Metric, symbol Device:C
- removed D? (x10): D_Schottky, Diode_SMD:D_SMC, symbol Device:D_Schottky
- removed J?: Screw_Terminal_01x04, TerminalBlock:TerminalBlock_bornier-4_P5.08mm, symbol Connector:Screw_Terminal_01x04
- removed J? (x5): Screw_Terminal_01x02, TerminalBlock:TerminalBlock_bornier-2_P5.08mm, symbol Connector:Screw_Terminal_01x02
- removed L? (x5): 22mkH, Inductor_SMD:L_10.4x10.4_H4.8, symbol Device:L_Small
- removed R? (x10): 1K, Resistor_SMD:R_0805_2012Metric, symbol Device:R
- removed R? (x50): 1R, Resistor_SMD:R_1206_3216Metric, symbol Device:R
- removed R? (x5): 100, Resistor_SMD:R_0805_2012Metric, symbol Device:R
- removed R? (x5): 100K, Resistor_SMD:R_0805_2012Metric, symbol Device:R
- removed U? (x5): LM3406, Package_SO:TSSOP-14-1EP_4.4x5mm_P0.65mm, symbol Regulator_Switching:LM3406
- added C1, C10, C100, C101, C103, C105, C107, C109, C11, C111, C113, C115, C117, C119, C121, C122, C123, C124, C125, C127, C128, C13, C130, C131, C133, C134, C136, C137, C139, C14, C140, C141, C143, C145, C147, C149, C151, C153, C155, C157, C159, C16, C161, C162, C163, C164, C165, C167, C168, C17, C170, C171, C173, C174, C176, C177, C179, C180, C181, C183, C185, C187, C189, C19, C191, C193, C195, C197, C199, C2, C20, C201, C209, C21, C213, C220, C23, C25, C27, C29, C3, C31, C33, C35, C37, C39, C4, C41, C42, C43, C44, C45, C47, C48, C5, C50, C51, C53, C54, C56, C57, C59, C60, C61, C63, C65, C67, C69, C7, C71, C73, C75, C77, C79, C8, C81, C82, C83, C84, C85, C87, C88, C90, C91, C93, C94, C96, C97, C99: 0.1mkF, Capacitor_SMD:C_0805_2012Metric, symbol Device:C
- added C102, C104, C106, C108, C110, C12, C126, C129, C132, C135, C138, C142, C144, C146, C148, C15, C150, C166, C169, C172, C175, C178, C18, C182, C184, C186, C188, C190, C22, C24, C26, C28, C30, C46, C49, C52, C55, C58, C6, C62, C64, C66, C68, C70, C86, C89, C9, C92, C95, C98: 470mkF, Capacitor_THT:CP_Radial_D10.0mm_P5.00mm, symbol Device:CP
- added C112, C114, C116, C118, C120, C152, C154, C156, C158, C160, C192, C194, C196, C198, C200, C32, C34, C36, C38, C40, C72, C74, C76, C78, C80: 1mkF, Capacitor_SMD:C_0805_2012Metric, symbol Device:C
- added C202, C203, C204, C205, C206, C207, C208, C212, C215: 0.1uf, Capacitor_SMD:C_0603_1608Metric, symbol Device:C
- added C210, C211: 18pF, Capacitor_SMD:C_0603_1608Metric, symbol Device:C
- added C214: 100uf 16v, Capacitor_THT:CP_Radial_D10.0mm_P5.00mm, symbol Device:CP_Small
- added C216: 10uf 10v, Capacitor_Tantalum_SMD:CP_EIA-3528-21_Kemet-B, symbol Device:C
- added C217, C218, C223: 0.1 mkf, Capacitor_SMD:C_0603_1608Metric_Pad1.05x0.95mm_HandSolder, symbol Device:C
- added C219: 220uf 50v, Capacitor_THT:CP_Radial_D10.0mm_P5.00mm, symbol Device:CP_Small
- added C221: 470uf 50v, Capacitor_THT:CP_Radial_D10.0mm_P5.00mm, symbol Device:CP_Small
- added C222: 10 mkf, Capacitor_SMD:C_0805_2012Metric_Pad1.15x1.40mm_HandSolder, symbol Device:C
- added D1, D10, D102, D2, D21, D22, D23, D24, D25, D26, D27, D28, D29, D3, D30, D4, D41, D42, D43, D44, D45, D46, D47, D48, D49, D5, D50, D6, D61, D62, D63, D64, D65, D66, D67, D68, D69, D7, D70, D8, D81, D82, D83, D84, D85, D86, D87, D88, D89, D9, D90: D_Schottky, Diode_SMD:D_SMC, symbol Device:D_Schottky
- added D100, D16, D17, D18, D19, D20, D36, D37, D38, D39, D40, D56, D57, D58, D59, D60, D76, D77, D78, D79, D80, D96, D97, D98, D99: lmc7101, Package_TO_SOT_SMD:SOT-23-5, symbol Amplifier_Operational:lmc7101
- added D101: AM1DS-0505S-NZ, Converter_DCDC:Converter_DCDC_muRata_NMAxxxxSC_THT, symbol Converter_DCDC:AM1DS-xxxxS-NZ
- added D103: Led_RGB_CA_2, LED_SMD:LED_Avago_PLCC4_3.2x2.8mm_CW, symbol Device:Led_RGB_CA_2
- added D104: SM712, Package_TO_SOT_SMD:SOT-23, symbol Device:SM712
- added D105: B380R, Diode_SMD:Diode_Bridge_Vishay_DFS, symbol Diode_Bridge:B380R
- added D106: LED, LED_SMD:LED_0805_2012Metric, symbol Device:LED
- added D11, D12, D13, D14, D15, D31, D32, D33, D34, D35, D51, D52, D53, D54, D55, D71, D72, D73, D74, D75, D91, D92, D93, D94, D95: Si2300, Package_TO_SOT_SMD:SOT-23, symbol Transistor_FET:Si2300
- added J1, J2, J3, J4, J5: Screw_Terminal_01x04, TerminalBlock:TerminalBlock_bornier-4_P5.08mm, symbol Connector:Screw_Terminal_01x04
- added J10, J11, J12, J13, J14, J15, J16, J17, J18, J19, J20, J21, J22, J23, J24, J25, J26, J27, J28, J29, J30, J35, J6, J7, J8, J9: Screw_Terminal_01x02, TerminalBlock:TerminalBlock_bornier-2_P5.08mm, symbol Connector:Screw_Terminal_01x02
- added J31: SWD, Connector_PinHeader_2.54mm:PinHeader_1x05_P2.54mm_Vertical, symbol Connector:Conn_01x05_Male
- added J32, J33: RJ45_Shielded, Connector_RJ:RJ45_Ninigi_GE, symbol Connector:RJ45_Shielded
- added J34: DEBUG, Connector_PinHeader_2.54mm:PinHeader_1x04_P2.54mm_Vertical, symbol Connector:Conn_01x04_Male
- added JP1: TX_UA, Jumper:SolderJumper-2_P1.3mm_Bridged_RoundedPad1.0x1.5mm, symbol Jumper:SolderJumper_2_Bridged
- added JP2: RX_UA, Jumper:SolderJumper-2_P1.3mm_Bridged_RoundedPad1.0x1.5mm, symbol Jumper:SolderJumper_2_Bridged
- added JP3: TX_CAN, Jumper:SolderJumper-2_P1.3mm_Open_RoundedPad1.0x1.5mm, symbol Jumper:SolderJumper_2_Open
- added JP4: RX_CAN, Jumper:SolderJumper-2_P1.3mm_Open_RoundedPad1.0x1.5mm, symbol Jumper:SolderJumper_2_Open
- added L1, L10, L11, L12, L13, L14, L15, L16, L17, L18, L19, L2, L20, L21, L22, L23, L24, L25, L3, L4, L5, L6, L7, L8, L9: 22mkH, Inductor_SMD:L_10.4x10.4_H4.8, symbol Device:L_Small
- added L26: 22 uH, Inductor_THT:L_Radial_D9.5mm_P5.00mm_Fastron_07HVP, symbol Device:INDUCTOR_SMALL
- added L27: 33 uH, Inductor_SMD:L_12x12mm_H8mm, symbol Device:INDUCTOR_SMALL
- added R1, R101, R102, R103, R104, R105, R11, R12, R13, R14, R15, R166, R167, R168, R169, R170, R171, R172, R173, R174, R175, R181, R182, R183, R184, R185, R191, R192, R193, R194, R195, R2, R256, R257, R258, R259, R260, R261, R262, R263, R264, R265, R271, R272, R273, R274, R275, R281, R282, R283, R284, R285, R3, R346, R347, R348, R349, R350, R351, R352, R353, R354, R355, R361, R362, R363, R364, R365, R371, R372, R373, R374, R375, R4, R436, R437, R438, R439, R440, R441, R442, R443, R444, R445, R455, R465, R5, R76, R77, R78, R79, R80, R81, R82, R83, R84, R85, R91, R92, R93, R94, R95: 1K, Resistor_SMD:R_0805_2012Metric, symbol Device:R
- added R10, R100, R161, R162, R163, R164, R165, R186, R187, R188, R189, R190, R251, R252, R253, R254, R255, R276, R277, R278, R279, R280, R341, R342, R343, R344, R345, R366, R367, R368, R369, R370, R431, R432, R433, R434, R435, R6, R7, R71, R72, R73, R74, R75, R8, R9, R96, R97, R98, R99: 100K, Resistor_SMD:R_0805_2012Metric, symbol Device:R
- added R106, R117, R128, R139, R150, R16, R196, R207, R218, R229, R240, R27, R286, R297, R308, R319, R330, R376, R38, R387, R398, R409, R420, R457, R49, R60: 100, Resistor_SMD:R_0805_2012Metric, symbol Device:R
- added R107, R108, R109, R110, R111, R112, R113, R114, R115, R116, R118, R119, R120, R121, R122, R123, R124, R125, R126, R127, R129, R130, R131, R132, R133, R134, R135, R136, R137, R138, R140, R141, R142, R143, R144, R145, R146, R147, R148, R149, R151, R152, R153, R154, R155, R156, R157, R158, R159, R160, R17, R18, R19, R197, R198, R199, R20, R200, R201, R202, R203, R204, R205, R206, R208, R209, R21, R210, R211, R212, R213, R214, R215, R216, R217, R219, R22, R220, R221, R222, R223, R224, R225, R226, R227, R228, R23, R230, R231, R232, R233, R234, R235, R236, R237, R238, R239, R24, R241, R242, R243, R244, R245, R246, R247, R248, R249, R25, R250, R26, R28, R287, R288, R289, R29, R290, R291, R292, R293, R294, R295, R296, R298, R299, R30, R300, R301, R302, R303, R304, R305, R306, R307, R309, R31, R310, R311, R312, R313, R314, R315, R316, R317, R318, R32, R320, R321, R322, R323, R324, R325, R326, R327, R328, R329, R33, R331, R332, R333, R334, R335, R336, R337, R338, R339, R34, R340, R35, R36, R37, R377, R378, R379, R380, R381, R382, R383, R384, R385, R386, R388, R389, R39, R390, R391, R392, R393, R394, R395, R396, R397, R399, R40, R400, R401, R402, R403, R404, R405, R406, R407, R408, R41, R410, R411, R412, R413, R414, R415, R416, R417, R418, R419, R42, R421, R422, R423, R424, R425, R426, R427, R428, R429, R43, R430, R44, R45, R46, R47, R48, R50, R51, R52, R53, R54, R55, R56, R57, R58, R59, R61, R62, R63, R64, R65, R66, R67, R68, R69, R70: 1R, Resistor_SMD:R_1206_3216Metric, symbol Device:R
- added R176, R177, R178, R179, R180, R266, R267, R268, R269, R270, R356, R357, R358, R359, R360, R446, R447, R448, R449, R450, R451, R453, R86, R87, R88, R89, R90: 10K, Resistor_SMD:R_0805_2012Metric, symbol Device:R
- added R452: 510, Resistor_SMD:R_0805_2012Metric, symbol Device:R
- added R454: 15, Resistor_SMD:R_1206_3216Metric, symbol Device:R
- added R456: 3K, Resistor_SMD:R_0805_2012Metric, symbol Device:R
- added R458, R460, R464, R469: 10k, Resistor_SMD:R_0805_2012Metric_Pad1.15x1.40mm_HandSolder, symbol Device:R
- added R459: 120 Om, Resistor_SMD:R_0805_2012Metric_Pad1.15x1.40mm_HandSolder, symbol Device:R
- added R461, R463: 10, Resistor_SMD:R_0805_2012Metric_Pad1.15x1.40mm_HandSolder, symbol Device:R
- added R462: 3.3k, Resistor_SMD:R_0805_2012Metric_Pad1.15x1.40mm_HandSolder, symbol Device:R
- added R466: 1.5k, Resistor_SMD:R_0805_2012Metric_Pad1.15x1.40mm_HandSolder, symbol Device:R
- added R467: 1k, Resistor_SMD:R_0805_2012Metric_Pad1.15x1.40mm_HandSolder, symbol Device:R
- added R468: 750 Om, Resistor_SMD:R_0805_2012Metric_Pad1.15x1.40mm_HandSolder, symbol Device:R
- added RV1: 10k, Potentiometer_THT:Potentiometer_Bourns_3296W_Vertical, symbol Device:POT
- added SW1: SW_DIP_x01, Button_Switch_THT:SW_DIP_SPSTx01_Slide_9.78x4.72mm_W7.62mm_P2.54mm, symbol Switch:SW_DIP_x01
- added TP1: A8, TestPoint:TestPoint_Pad_D1.0mm, symbol Connector:TestPoint
- added TP10: E7, TestPoint:TestPoint_Pad_D1.0mm, symbol Connector:TestPoint
- added TP11: E10, TestPoint:TestPoint_Pad_D1.0mm, symbol Connector:TestPoint
- added TP12: E12, TestPoint:TestPoint_Pad_D1.0mm, symbol Connector:TestPoint
- added TP13: B13, TestPoint:TestPoint_Pad_D1.0mm, symbol Connector:TestPoint
- added TP14: C4, TestPoint:TestPoint_Pad_D1.0mm, symbol Connector:TestPoint
- added TP15: C5, TestPoint:TestPoint_Pad_D1.0mm, symbol Connector:TestPoint
- added TP16: C13, TestPoint:TestPoint_Pad_D1.0mm, symbol Connector:TestPoint
- added TP17: C14, TestPoint:TestPoint_Pad_D1.0mm, symbol Connector:TestPoint
- added TP18: C15, TestPoint:TestPoint_Pad_D1.0mm, symbol Connector:TestPoint
- added TP2: REF, TestPoint:TestPoint_Pad_D1.0mm, symbol Connector:TestPoint
- added TP3: F6, TestPoint:TestPoint_Pad_D1.0mm, symbol Connector:TestPoint
- added TP4: B0, TestPoint:TestPoint_Pad_D1.0mm, symbol Connector:TestPoint
- added TP5: E1, TestPoint:TestPoint_Pad_D1.0mm, symbol Connector:TestPoint
- added TP6: B1, TestPoint:TestPoint_Pad_D1.0mm, symbol Connector:TestPoint
- added TP7: B2, TestPoint:TestPoint_Pad_D1.0mm, symbol Connector:TestPoint
- added TP8: E6, TestPoint:TestPoint_Pad_D1.0mm, symbol Connector:TestPoint
- added TP9: GND, TestPoint:TestPoint_Pad_D1.0mm, symbol Connector:TestPoint
- added U1, U10, U11, U12, U13, U14, U15, U16, U17, U18, U19, U2, U20, U21, U22, U23, U24, U25, U3, U4, U5, U6, U7, U8, U9: LM3406, Package_SO:TSSOP-14-1EP_4.4x5mm_P0.65mm, symbol Regulator_Switching:LM3406
- added U26, U27, U32, U37: 74HC595, Package_SO:SOP-16_4.55x10.3mm_P1.27mm, symbol 74xx:74HC595
- added U28: TL431LP, Package_TO_SOT_THT:TO-92_Inline, symbol Reference_Voltage:TL431LP
- added U30: MCP2551-I_SN, Package_SO:SO-8_3.9x4.9mm_P1.27mm, symbol Interface:MCP2551-I_SN
- added U31: LM1117-3.3, Package_TO_SOT_THT:TO-220-3_Vertical, symbol Regulator_Linear:LM1117-3.3
- added U33: GD25Q16C, Package_SO:PowerIntegrations_SO-8, symbol Memory_Flash:GD25Q16C
- added U34: MAX3485, Package_SO:SOIC-8_3.9x4.9mm_P1.27mm, symbol Interface_UART:MAX3485
- added U35: ISO7341C, Package_SO:SOIC-16W_7.5x10.3mm_P1.27mm, symbol Isolator:ISO7341C
- added U36: LM2596S-ADJ, Package_TO_SOT_SMD:TO-263-5_TabPin3, symbol Regulator_Switching:LM2596S-ADJ
- added Y1: Crystal_Small, Crystal:Crystal_SMD_HC49-SD, symbol Device:Crystal_Small
- gave numbers to parts that had none: 1
Connections:
- net GND: now also U29.20 (VSSA), U29.49 (VSS), U29.74 (VSS), U29.99 (VSS), C10.2, C100.2, C11.2, C111.2, C112.2, C113.2, C114.2, C115.2, C116.2, C117.2, C118.2, C119.2, C12.2, C120.2, C126.2, C127.2, C128.2, C129.2, C13.2, C130.2, C131.2, C132.2, C133.2, C134.2, C135.2, C136.2, C137.2, C138.2, C139.2, C14.2, C140.2, C15.2, C151.2, C152.2, C153.2, C154.2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
- net DIM_CH6: now reaches U29.1 (PE2)
- net DIM_CH6: now also R27.2
- net DIM_CH10: now reaches U29.10 (PF9)
- net DIM_CH10: now also R387.2
- net +3V3: now reaches U29.100 (VDD)
- net +3V3: now also U29.22 (VDDA), U29.28 (VDD), U29.50 (VDD), U29.6 (VBAT), U29.75 (VDD), C201.1, C202.1, C203.1, C204.1, C205.1, C206.1, C207.1, C209.1, C212.2, C213.1, C215.1, C216.1, C217.2, C220.1, D100.2 (V+), D103.4, D16.2 (V+), D17.2 (V+), D18.2 (V+), D19.2 (V+), D20.2 (V+), D36.2 (V+), D37.2 (V+), D38.2 (V+), D39.2 (V+), D40.2 (V+), D56.2 (V+), D57.2 (V+), D58.2 (V+), D59.2 (V+), D60.2 (V+), D76.2 (V+), D77.2 (V+), D78.2 (V+), D79.2 (V+)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
- net DIM_CH11: now reaches U29.11 (PF10)
- net DIM_CH11: now also R38.2
- net at U29.12 (PF0): now also C210.1, Y1.1
- net at U29.13 (PF1): now also C211.2, Y1.2
- net RESET: now reaches U29.14 (NRST)
- net RESET: now also C208.2, J31.1 (Pin_1), R453.1
- net Isens_CH1: now reaches U29.15 (PC0)
- net Isens_CH1: now also D16.1, R86.2
- net Isens_CH2: now reaches U29.16 (PC1)
- net Isens_CH2: now also D36.1, R176.2
- net Isens_CH3: now reaches U29.17 (PC2)
- net Isens_CH3: now also D56.1, R266.2
- net Isens_CH4: now reaches U29.18 (PC3)
- net Isens_CH4: now also D76.1, R356.2
- net Isens_CH5: now reaches U29.19 (PF2)
- net Isens_CH5: now also D96.1, R446.2
- net DIM_CH7: now reaches U29.2 (PE3)
- net DIM_CH7: now also R117.2
- net at U29.21 (VREF+): now also R454.1, R455.2, TP2.1, U28.3 (K)
- net Isens_CH6: now reaches U29.23 (PA0)
- net Isens_CH6: now also D17.1, R87.2
- net Isens_CH7: now reaches U29.24 (PA1)
- net Isens_CH7: now also D37.1, R177.2
- net Isens_CH8: now reaches U29.25 (PA2)
- net Isens_CH8: now also D57.1, R267.2
- net Isens_CH9: now reaches U29.26 (PA3)
- net Isens_CH9: now also D77.1, R357.2
- net Isens_CH10: now reaches U29.27 (PF4)
- net Isens_CH10: now also D97.1, R447.2
- net Isens_CH11: now reaches U29.29 (PA4)
- net Isens_CH11: now also D18.1, R88.2
- net DIM_CH8: now reaches U29.3 (PE4)
- net DIM_CH8: now also R207.2
- net Isens_CH12: now reaches U29.30 (PA5)
- net Isens_CH12: now also D38.1, R178.2
- net DIM_CH12: now reaches U29.31 (PA6)
- net DIM_CH12: now also R128.2
- net DIM_CH13: now reaches U29.32 (PA7)
- net DIM_CH13: now also R218.2
- net at U29.33 (PC4): now also TP14.1
- net at U29.34 (PC5): now also TP15.1
- net at U29.35 (PB0): now also TP4.1
- net at U29.36 (PB1): now also TP6.1
- net at U29.37 (PB2): now also TP7.1
- net at U29.38 (PE7): now also TP10.1
- net Isens_CH13: now reaches U29.39 (PE8)
- net Isens_CH13: now also D58.1, R268.2
- net DIM_CH9: now reaches U29.4 (PE5)
- net DIM_CH9: now also R297.2
- net DIM_CH14: now reaches U29.40 (PE9)
- net DIM_CH14: now also R308.2
- net at U29.41 (PE10): now also TP11.1
- net DIM_CH15: now reaches U29.42 (PE11)
- net DIM_CH15: now also R398.2
- net at U29.43 (PE12): now also TP12.1
- net DIM_CH16: now reaches U29.44 (PE13)
- net DIM_CH16: now also R49.2
- net Isens_CH14: now reaches U29.45 (PE14)
- net Isens_CH14: now also D78.1, R358.2
- net Isens_CH15: now reaches U29.46 (PE15)
- net Isens_CH15: now also D98.1, R448.2
- net DIM_CH17: now reaches U29.47 (PB10)
- net DIM_CH17: now also R139.2
- net DIM_CH18: now reaches U29.48 (PB11)
- net DIM_CH18: now also R229.2
- net at U29.5 (PE6): now also TP8.1
- net Isens_CH16: now reaches U29.51 (PB12)
- net Isens_CH16: now also D19.1, R89.2
- net at U29.52 (PB13): now also TP13.1
- net Isens_CH17: now reaches U29.53 (PB14)
- net Isens_CH17: now also D39.1, R179.2
- net Isens_CH18: now reaches U29.54 (PB15)
- net Isens_CH18: now also D59.1, R269.2
- net Isens_CH19: now reaches U29.55 (PD8)
- net Isens_CH19: now also D79.1, R359.2
- net Isens_CH20: now reaches U29.56 (PD9)
- net Isens_CH20: now also D99.1, R449.2
- net Isens_CH21: now reaches U29.57 (PD10)
- net Isens_CH21: now also D20.1, R90.2
- net Isens_CH22: now reaches U29.58 (PD11)
- net Isens_CH22: now also D40.1, R180.2
- net Isens_CH23: now reaches U29.59 (PD12)
- net Isens_CH23: now also D60.1, R270.2
- net Isens_CH24: now reaches U29.60 (PD13)
- net Isens_CH24: now also D80.1, R360.2
- net Isens_CH25: now reaches U29.61 (PD14)
- net Isens_CH25: now also D100.1, R450.2
- net DIM_CH19: now reaches U29.62 (PD15)
- net DIM_CH19: now also R319.2
- net DIM_CH20: now reaches U29.63 (PC6)
- net DIM_CH20: now also R409.2
- net DIM_CH21: now reaches U29.64 (PC7)
- net DIM_CH21: now also R60.2
- net DIM_CH22: now reaches U29.65 (PC8)
- net DIM_CH22: now also R150.2
- net DIM_CH23: now reaches U29.66 (PC9)
- net DIM_CH23: now also R240.2
- net at U29.67 (PA8): now also TP1.1
- net at U29.68 (PA9): now also JP1.1 (A)
- net at U29.69 (PA10): now also JP2.1 (A)
- net at U29.7 (PC13): now also TP16.1
- net DIM_CH24: now reaches U29.70 (PA11)
- net DIM_CH24: now also R330.2, R420.2
- net DE: now reaches U29.71 (PA12)
- net DE: now also U35.4 (INB)
- net SWDIO: now reaches U29.72 (PA13)
- net SWDIO: now also J31.2 (Pin_2)
- net at U29.73 (PF6): now also TP3.1
- net SWDCL: now reaches U29.76 (PA14)
- net SWDCL: now also J31.4 (Pin_4)
- net spi_CS: now reaches U29.77 (PA15)
- net spi_CS: now also U26.12 (RCLK), U27.12 (RCLK), U32.12 (RCLK), U37.12 (RCLK)
- net SPI3_CLK: now reaches U29.78 (PC10)
- net SPI3_CLK: now also U33.6 (CLK)
- net SPI3_MISO: now reaches U29.79 (PC11)
- net SPI3_MISO: now also U33.2 (DO(IO1))
- net at U29.8 (PC14): now also TP17.1
- net SPI3_MOSI: now reaches U29.80 (PC12)
- net SPI3_MOSI: now also U33.5 (DI(IO0))
- net at U29.81 (PD0): now also JP3.2 (B)
- net at U29.82 (PD1): now also JP4.2 (B)
- net SPI3_CS: now reaches U29.83 (PD2)
- net SPI3_CS: now also U33.1 (~CS)
- net DIM_CH1: now reaches U29.84 (PD3)
- net DIM_CH1: now also R16.2
- net DIM_CH2: now reaches U29.85 (PD4)
- net DIM_CH2: now also R106.2
- net USART2_TX: now reaches U29.86 (PD5)
- net USART2_TX: now also J34.1 (Pin_1)
- net USART2_RX: now reaches U29.87 (PD6)
- net USART2_RX: now also J34.3 (Pin_3)
- net ~OE: now reaches U29.88 (PD7)
- net ~OE: now also U26.13 (G), U27.13 (G), U32.13 (G), U37.13 (G)
- net spi_SCK: now reaches U29.89 (PB3)
- net spi_SCK: now also U26.11 (SRCLK), U27.11 (SRCLK), U32.11 (SRCLK), U37.11 (SRCLK)
- net at U29.9 (PC15): now also TP18.1
- net ~MR: now reaches U29.90 (PB4)
- net ~MR: now also U26.10 (SRCLR), U27.10 (SRCLR), U32.10 (SRCLR), U37.10 (SRCLR)
- net spi_MOSI: now reaches U29.91 (PB5)
- net spi_MOSI: now also U26.14 (SER)
- net DIM_CH3: now reaches U29.92 (PB6)
- net DIM_CH3: now also R196.2
- net DIM_CH4: now reaches U29.93 (PB7)
- net DIM_CH4: now also R286.2
- net at U29.94 (BOOT0): now also R451.1, R452.1
- net DIM_CH5: now reaches U29.95 (PB8)
- net DIM_CH5: now also R376.2
- net SPI3_HOLD: now reaches U29.96 (PB9)
- net SPI3_HOLD: now also U33.7 (~HOLD)
- net SPI3_WP: now reaches U29.97 (PE0)
- net SPI3_WP: now also U33.3 (~WP)
- net at U29.98 (PE1): now also TP5.1
- new net: C4.1, D4.1 (K), L4.1, U4.1 (SW), U4.2 (SW)
- new net: R9.1, U4.10 (RON)
- new net: C38.1, U4.11 (VCC)
- new net: C135.1, C136.1, C137.1, C15.1, C16.1, C17.1, C175.1, C176.1, C177.1, C55.1, C56.1, C57.1, C95.1, C96.1, C97.1, D14.3 (D), D29.1 (K), D34.3 (D), D49.1 (K), D54.3 (D), D69.1 (K), D74.3 (D), D89.1 (K), D9.1 (K), D94.3 (D), J4.3 (Pin_3), J4.4 (Pin_4), R189.2, R279.2, R369.2, R9.2, R99.2, U14.12 (VINS), U14.13 (VIN), U14.14 (VIN), U19.12 (VINS), U19.13 (VIN), U19.14 (VIN), U24.12 (VINS), U24.13 (VIN)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
- new net: C4.2, U4.3 (BOOT)
- new net: R4.2, U4.5 (VOUT)
- new net: R14.2, U4.6 (CS)
- new net: R49.1, U4.8 (DIM)
- new net: C37.1, U4.9 (COMP)
- new net: C27.1, C28.1, D9.2 (A), J9.1 (Pin_1), L4.2, R4.1
- new net: C27.2, C28.2, J9.2 (Pin_2), R14.1, R50.2, R51.2, R52.2, R53.2, R54.2, R55.2, R56.2, R57.2, R58.2, R59.2, R79.1
- new net: D19.3 (+), R79.2
- new net: D19.4 (-), R84.2, R89.1
- new net: C44.1, D24.1 (K), L9.1, U9.1 (SW), U9.2 (SW)
- new net: R99.1, U9.10 (RON)
- new net: C78.1, U9.11 (VCC)
- new net: C44.2, U9.3 (BOOT)
- new net: R94.2, U9.5 (VOUT)
- new net: R104.2, U9.6 (CS)
- new net: R139.1, U9.8 (DIM)
- new net: C77.1, U9.9 (COMP)
- new net: C67.1, C68.1, D29.2 (A), J14.1 (Pin_1), L9.2, R94.1
- new net: C67.2, C68.2, J14.2 (Pin_2), R104.1, R140.2, R141.2, R142.2, R143.2, R144.2, R145.2, R146.2, R147.2, R148.2, R149.2, R169.1
- new net: D39.3 (+), R169.2
- new net: D39.4 (-), R174.2, R179.1
- new net: C84.1, D44.1 (K), L14.1, U14.1 (SW), U14.2 (SW)
- new net: R189.1, U14.10 (RON)
- new net: C118.1, U14.11 (VCC)
- new net: C84.2, U14.3 (BOOT)
- new net: R184.2, U14.5 (VOUT)
- new net: R194.2, U14.6 (CS)
- new net: R229.1, U14.8 (DIM)
- new net: C117.1, U14.9 (COMP)
- new net: C107.1, C108.1, D49.2 (A), J19.1 (Pin_1), L14.2, R184.1
- new net: C107.2, C108.2, J19.2 (Pin_2), R194.1, R230.2, R231.2, R232.2, R233.2, R234.2, R235.2, R236.2, R237.2, R238.2, R239.2, R259.1
- new net: D59.3 (+), R259.2
- new net: D59.4 (-), R264.2, R269.1
- new net: C124.1, D64.1 (K), L19.1, U19.1 (SW), U19.2 (SW)
- new net: R279.1, U19.10 (RON)
- new net: C158.1, U19.11 (VCC)
- new net: C124.2, U19.3 (BOOT)
- new net: R274.2, U19.5 (VOUT)
- new net: R284.2, U19.6 (CS)
- new net: R319.1, U19.8 (DIM)
- new net: C157.1, U19.9 (COMP)
- new net: C147.1, C148.1, D69.2 (A), J24.1 (Pin_1), L19.2, R274.1
- new net: C147.2, C148.2, J24.2 (Pin_2), R284.1, R320.2, R321.2, R322.2, R323.2, R324.2, R325.2, R326.2, R327.2, R328.2, R329.2, R349.1
- new net: D79.3 (+), R349.2
- new net: D79.4 (-), R354.2, R359.1
- new net: C164.1, D84.1 (K), L24.1, U24.1 (SW), U24.2 (SW)
- new net: R369.1, U24.10 (RON)
- new net: C198.1, U24.11 (VCC)
- new net: C164.2, U24.3 (BOOT)
- new net: R364.2, U24.5 (VOUT)
- new net: R374.2, U24.6 (CS)
- new net: R409.1, U24.8 (DIM)
- new net: C197.1, U24.9 (COMP)
- new net: C187.1, C188.1, D89.2 (A), J29.1 (Pin_1), L24.2, R364.1
- new net: C187.2, C188.2, J29.2 (Pin_2), R374.1, R410.2, R411.2, R412.2, R413.2, R414.2, R415.2, R416.2, R417.2, R418.2, R419.2, R439.1
- new net: D99.3 (+), R439.2
- new net: D99.4 (-), R444.2, R449.1
- new net: C214.1, L26.2, R454.2, U31.3 (VI)
- new net: C3.1, D3.1 (K), L3.1, U3.1 (SW), U3.2 (SW)
- new net: R8.1, U3.10 (RON)
- new net: C36.1, U3.11 (VCC)
- new net: C12.1, C13.1, C132.1, C133.1, C134.1, C14.1, C172.1, C173.1, C174.1, C52.1, C53.1, C54.1, C92.1, C93.1, C94.1, D13.3 (D), D28.1 (K), D33.3 (D), D48.1 (K), D53.3 (D), D68.1 (K), D73.3 (D), D8.1 (K), D88.1 (K), D93.3 (D), J3.3 (Pin_3), J3.4 (Pin_4), R188.2, R278.2, R368.2, R8.2, R98.2, U13.12 (VINS), U13.13 (VIN), U13.14 (VIN), U18.12 (VINS), U18.13 (VIN), U18.14 (VIN), U23.12 (VINS), U23.13 (VIN)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
- new net: C3.2, U3.3 (BOOT)
- new net: R3.2, U3.5 (VOUT)
- new net: R13.2, U3.6 (CS)
- new net: R38.1, U3.8 (DIM)
- new net: C35.1, U3.9 (COMP)
- new net: C25.1, C26.1, D8.2 (A), J8.1 (Pin_1), L3.2, R3.1
- new net: C25.2, C26.2, J8.2 (Pin_2), R13.1, R39.2, R40.2, R41.2, R42.2, R43.2, R44.2, R45.2, R46.2, R47.2, R48.2, R78.1
- new net: D18.3 (+), R78.2
- new net: D18.4 (-), R83.2, R88.1
- new net: C43.1, D23.1 (K), L8.1, U8.1 (SW), U8.2 (SW)
- new net: R98.1, U8.10 (RON)
- new net: C76.1, U8.11 (VCC)
- new net: C43.2, U8.3 (BOOT)
- new net: R93.2, U8.5 (VOUT)
- new net: R103.2, U8.6 (CS)
- new net: R128.1, U8.8 (DIM)
- new net: C75.1, U8.9 (COMP)
- new net: C65.1, C66.1, D28.2 (A), J13.1 (Pin_1), L8.2, R93.1
- new net: C65.2, C66.2, J13.2 (Pin_2), R103.1, R129.2, R130.2, R131.2, R132.2, R133.2, R134.2, R135.2, R136.2, R137.2, R138.2, R168.1
- new net: D38.3 (+), R168.2
- new net: D38.4 (-), R173.2, R178.1
- new net: C83.1, D43.1 (K), L13.1, U13.1 (SW), U13.2 (SW)
- new net: R188.1, U13.10 (RON)
- new net: C116.1, U13.11 (VCC)
- new net: C83.2, U13.3 (BOOT)
- new net: R183.2, U13.5 (VOUT)
- new net: R193.2, U13.6 (CS)
- new net: R218.1, U13.8 (DIM)
- new net: C115.1, U13.9 (COMP)
- new net: C105.1, C106.1, D48.2 (A), J18.1 (Pin_1), L13.2, R183.1
- new net: C105.2, C106.2, J18.2 (Pin_2), R193.1, R219.2, R220.2, R221.2, R222.2, R223.2, R224.2, R225.2, R226.2, R227.2, R228.2, R258.1
- new net: D58.3 (+), R258.2
- new net: D58.4 (-), R263.2, R268.1
- new net: C123.1, D63.1 (K), L18.1, U18.1 (SW), U18.2 (SW)
- new net: R278.1, U18.10 (RON)
- new net: C156.1, U18.11 (VCC)
- new net: C123.2, U18.3 (BOOT)
- new net: R273.2, U18.5 (VOUT)
- new net: R283.2, U18.6 (CS)
- new net: R308.1, U18.8 (DIM)
- new net: C155.1, U18.9 (COMP)
- new net: C145.1, C146.1, D68.2 (A), J23.1 (Pin_1), L18.2, R273.1
- new net: C145.2, C146.2, J23.2 (Pin_2), R283.1, R309.2, R310.2, R311.2, R312.2, R313.2, R314.2, R315.2, R316.2, R317.2, R318.2, R348.1
- new net: D78.3 (+), R348.2
- new net: D78.4 (-), R353.2, R358.1
- new net: C163.1, D83.1 (K), L23.1, U23.1 (SW), U23.2 (SW)
- new net: R368.1, U23.10 (RON)
- new net: C196.1, U23.11 (VCC)
- new net: C163.2, U23.3 (BOOT)
- new net: R363.2, U23.5 (VOUT)
- new net: R373.2, U23.6 (CS)
- new net: R398.1, U23.8 (DIM)
- new net: C195.1, U23.9 (COMP)
- new net: C185.1, C186.1, D88.2 (A), J28.1 (Pin_1), L23.2, R363.1
- new net: C185.2, C186.2, J28.2 (Pin_2), R373.1, R399.2, R400.2, R401.2, R402.2, R403.2, R404.2, R405.2, R406.2, R407.2, R408.2, R438.1
- new net: D98.3 (+), R438.2
- new net: D98.4 (-), R443.2, R448.1
- new net: U26.9 (~QH), U27.14 (SER)
- new net: U27.9 (~QH), U32.14 (SER)
- new net: C2.1, D2.1 (K), L2.1, U2.1 (SW), U2.2 (SW)
- new net: R7.1, U2.10 (RON)
- new net: C34.1, U2.11 (VCC)
- new net: C10.1, C11.1, C129.1, C130.1, C131.1, C169.1, C170.1, C171.1, C49.1, C50.1, C51.1, C89.1, C9.1, C90.1, C91.1, D12.3 (D), D27.1 (K), D32.3 (D), D47.1 (K), D52.3 (D), D67.1 (K), D7.1 (K), D72.3 (D), D87.1 (K), D92.3 (D), J2.3 (Pin_3), J2.4 (Pin_4), R187.2, R277.2, R367.2, R7.2, R97.2, U12.12 (VINS), U12.13 (VIN), U12.14 (VIN), U17.12 (VINS), U17.13 (VIN), U17.14 (VIN), U2.12 (VINS), U2.13 (VIN)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
- new net: C2.2, U2.3 (BOOT)
- new net: R2.2, U2.5 (VOUT)
- new net: R12.2, U2.6 (CS)
- new net: R27.1, U2.8 (DIM)
- new net: C33.1, U2.9 (COMP)
- new net: C23.1, C24.1, D7.2 (A), J7.1 (Pin_1), L2.2, R2.1
- new net: C23.2, C24.2, J7.2 (Pin_2), R12.1, R28.2, R29.2, R30.2, R31.2, R32.2, R33.2, R34.2, R35.2, R36.2, R37.2, R77.1
- new net: D17.3 (+), R77.2
- new net: D17.4 (-), R82.2, R87.1
- new net: C42.1, D22.1 (K), L7.1, U7.1 (SW), U7.2 (SW)
- new net: R97.1, U7.10 (RON)
- new net: C74.1, U7.11 (VCC)
- new net: C42.2, U7.3 (BOOT)
- new net: R92.2, U7.5 (VOUT)
- new net: R102.2, U7.6 (CS)
- new net: R117.1, U7.8 (DIM)
- new net: C73.1, U7.9 (COMP)
- new net: C63.1, C64.1, D27.2 (A), J12.1 (Pin_1), L7.2, R92.1
- new net: C63.2, C64.2, J12.2 (Pin_2), R102.1, R118.2, R119.2, R120.2, R121.2, R122.2, R123.2, R124.2, R125.2, R126.2, R127.2, R167.1
- new net: D37.3 (+), R167.2
- new net: D37.4 (-), R172.2, R177.1
- new net: C82.1, D42.1 (K), L12.1, U12.1 (SW), U12.2 (SW)
- new net: R187.1, U12.10 (RON)
- new net: C114.1, U12.11 (VCC)
- new net: C82.2, U12.3 (BOOT)
- new net: R182.2, U12.5 (VOUT)
- new net: R192.2, U12.6 (CS)
- new net: R207.1, U12.8 (DIM)
- new net: C113.1, U12.9 (COMP)
- new net: C103.1, C104.1, D47.2 (A), J17.1 (Pin_1), L12.2, R182.1
- new net: C103.2, C104.2, J17.2 (Pin_2), R192.1, R208.2, R209.2, R210.2, R211.2, R212.2, R213.2, R214.2, R215.2, R216.2, R217.2, R257.1
- new net: D57.3 (+), R257.2
- new net: D57.4 (-), R262.2, R267.1
- new net: C122.1, D62.1 (K), L17.1, U17.1 (SW), U17.2 (SW)
- new net: R277.1, U17.10 (RON)
- new net: C154.1, U17.11 (VCC)
- new net: C122.2, U17.3 (BOOT)
- new net: R272.2, U17.5 (VOUT)
- new net: R282.2, U17.6 (CS)
- new net: R297.1, U17.8 (DIM)
- new net: C153.1, U17.9 (COMP)
- new net: C143.1, C144.1, D67.2 (A), J22.1 (Pin_1), L17.2, R272.1
- new net: C143.2, C144.2, J22.2 (Pin_2), R282.1, R298.2, R299.2, R300.2, R301.2, R302.2, R303.2, R304.2, R305.2, R306.2, R307.2, R347.1
- new net: D77.3 (+), R347.2
- new net: D77.4 (-), R352.2, R357.1
- new net: C162.1, D82.1 (K), L22.1, U22.1 (SW), U22.2 (SW)
- new net: R367.1, U22.10 (RON)
- new net: C194.1, U22.11 (VCC)
- new net: C162.2, U22.3 (BOOT)
- new net: R362.2, U22.5 (VOUT)
- new net: R372.2, U22.6 (CS)
- new net: R387.1, U22.8 (DIM)
- new net: C193.1, U22.9 (COMP)
- new net: C183.1, C184.1, D87.2 (A), J27.1 (Pin_1), L22.2, R362.1
- new net: C183.2, C184.2, J27.2 (Pin_2), R372.1, R388.2, R389.2, R390.2, R391.2, R392.2, R393.2, R394.2, R395.2, R396.2, R397.2, R437.1
- new net: D97.3 (+), R437.2
- new net: D97.4 (-), R442.2, R447.1
- new net: D102.1 (K), L27.1, U36.2 (OUT)
- new net: R462.1, R465.2, U36.4 (FB)
- new net: U32.9 (~QH), U37.14 (SER)
- new net: C1.1, D1.1 (K), L1.1, U1.1 (SW), U1.2 (SW)
- new net: R6.1, U1.10 (RON)
- new net: C32.1, U1.11 (VCC)
- new net: C126.1, C127.1, C128.1, C166.1, C167.1, C168.1, C46.1, C47.1, C48.1, C6.1, C7.1, C8.1, C86.1, C87.1, C88.1, D11.3 (D), D26.1 (K), D31.3 (D), D46.1 (K), D51.3 (D), D6.1 (K), D66.1 (K), D71.3 (D), D86.1 (K), D91.3 (D), J1.3 (Pin_3), J1.4 (Pin_4), R186.2, R276.2, R366.2, R6.2, R96.2, U1.12 (VINS), U1.13 (VIN), U1.14 (VIN), U11.12 (VINS), U11.13 (VIN), U11.14 (VIN), U16.12 (VINS), U16.13 (VIN)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
- new net: C1.2, U1.3 (BOOT)
- new net: R1.2, U1.5 (VOUT)
- new net: R11.2, U1.6 (CS)
- new net: R16.1, U1.8 (DIM)
- new net: C31.1, U1.9 (COMP)
- new net: C21.1, C22.1, D6.2 (A), J6.1 (Pin_1), L1.2, R1.1
- new net: C21.2, C22.2, J6.2 (Pin_2), R11.1, R17.2, R18.2, R19.2, R20.2, R21.2, R22.2, R23.2, R24.2, R25.2, R26.2, R76.1
- new net: D16.3 (+), R76.2
- new net: D16.4 (-), R81.2, R86.1
- new net: C41.1, D21.1 (K), L6.1, U6.1 (SW), U6.2 (SW)
- new net: R96.1, U6.10 (RON)
- new net: C72.1, U6.11 (VCC)
- new net: C41.2, U6.3 (BOOT)
- new net: R91.2, U6.5 (VOUT)
- new net: R101.2, U6.6 (CS)
- new net: R106.1, U6.8 (DIM)
- new net: C71.1, U6.9 (COMP)
- new net: C61.1, C62.1, D26.2 (A), J11.1 (Pin_1), L6.2, R91.1
- new net: C61.2, C62.2, J11.2 (Pin_2), R101.1, R107.2, R108.2, R109.2, R110.2, R111.2, R112.2, R113.2, R114.2, R115.2, R116.2, R166.1
- new net: D36.3 (+), R166.2
- new net: D36.4 (-), R171.2, R176.1
- new net: C81.1, D41.1 (K), L11.1, U11.1 (SW), U11.2 (SW)
- new net: R186.1, U11.10 (RON)
- new net: C112.1, U11.11 (VCC)
- new net: C81.2, U11.3 (BOOT)
- new net: R181.2, U11.5 (VOUT)
- new net: R191.2, U11.6 (CS)
- new net: R196.1, U11.8 (DIM)
- new net: C111.1, U11.9 (COMP)
- new net: C101.1, C102.1, D46.2 (A), J16.1 (Pin_1), L11.2, R181.1
- new net: C101.2, C102.2, J16.2 (Pin_2), R191.1, R197.2, R198.2, R199.2, R200.2, R201.2, R202.2, R203.2, R204.2, R205.2, R206.2, R256.1
- new net: D56.3 (+), R256.2
- new net: D56.4 (-), R261.2, R266.1
- new net: C121.1, D61.1 (K), L16.1, U16.1 (SW), U16.2 (SW)
- new net: R276.1, U16.10 (RON)
- new net: C152.1, U16.11 (VCC)
- new net: C121.2, U16.3 (BOOT)
- new net: R271.2, U16.5 (VOUT)
- new net: R281.2, U16.6 (CS)
- new net: R286.1, U16.8 (DIM)
- new net: C151.1, U16.9 (COMP)
- new net: C141.1, C142.1, D66.2 (A), J21.1 (Pin_1), L16.2, R271.1
- new net: C141.2, C142.2, J21.2 (Pin_2), R281.1, R287.2, R288.2, R289.2, R290.2, R291.2, R292.2, R293.2, R294.2, R295.2, R296.2, R346.1
- new net: D76.3 (+), R346.2
- new net: D76.4 (-), R351.2, R356.1
- new net: C161.1, D81.1 (K), L21.1, U21.1 (SW), U21.2 (SW)
- new net: R366.1, U21.10 (RON)
- new net: C192.1, U21.11 (VCC)
- new net: C161.2, U21.3 (BOOT)
- new net: R361.2, U21.5 (VOUT)
- new net: R371.2, U21.6 (CS)
- new net: R376.1, U21.8 (DIM)
- new net: C191.1, U21.9 (COMP)
- new net: C181.1, C182.1, D86.2 (A), J26.1 (Pin_1), L21.2, R361.1
- new net: C181.2, C182.2, J26.2 (Pin_2), R371.1, R377.2, R378.2, R379.2, R380.2, R381.2, R382.2, R383.2, R384.2, R385.2, R386.2, R436.1
- new net: D96.3 (+), R436.2
- new net: D96.4 (-), R441.2, R446.1
- new net: R459.2, SW1.1
- new net: D104.1, R463.1, U30.6 (CANL), U34.6 (A)
- new net: D104.2, R461.1, U30.7 (CANH), U34.7 (B)
- new net: D106.2 (A), R469.2
- new net: R458.2, U30.8 (Rs)
- new net: C5.1, D5.1 (K), L5.1, U5.1 (SW), U5.2 (SW)
- new net: R10.1, U5.10 (RON)
- new net: C40.1, U5.11 (VCC)
- new net: C100.1, C138.1, C139.1, C140.1, C178.1, C179.1, C18.1, C180.1, C19.1, C20.1, C58.1, C59.1, C60.1, C98.1, C99.1, D10.1 (K), D15.3 (D), D30.1 (K), D35.3 (D), D50.1 (K), D55.3 (D), D70.1 (K), D75.3 (D), D90.1 (K), D95.3 (D), J5.3 (Pin_3), J5.4 (Pin_4), R10.2, R100.2, R190.2, R280.2, R370.2, U10.12 (VINS), U10.13 (VIN), U10.14 (VIN), U15.12 (VINS), U15.13 (VIN), U15.14 (VIN), U20.12 (VINS), U20.13 (VIN)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
- new net: C5.2, U5.3 (BOOT)
- new net: R5.2, U5.5 (VOUT)
- new net: R15.2, U5.6 (CS)
- new net: R60.1, U5.8 (DIM)
- new net: C39.1, U5.9 (COMP)
- new net: C29.1, C30.1, D10.2 (A), J10.1 (Pin_1), L5.2, R5.1
- new net: C29.2, C30.2, J10.2 (Pin_2), R15.1, R61.2, R62.2, R63.2, R64.2, R65.2, R66.2, R67.2, R68.2, R69.2, R70.2, R80.1
- new net: R455.1, R456.2, RV1.1, RV1.2, U28.1 (REF)
- new net: C219.1, D101.1 (+VIN), L27.2, R462.2
- new net: D105.2 (~~), J35.1 (Pin_1)
- new net: D105.4 (~~), J35.2 (Pin_2)
- new net: D101.6 (+VOUT), L26.1
- new net: D103.1 (B), R466.2
- new net: D103.2 (G), R467.2
- new net: D103.3 (R), R468.2
- new net: D20.3 (+), R80.2
- new net: D20.4 (-), R85.2, R90.1
- new net: C45.1, D25.1 (K), L10.1, U10.1 (SW), U10.2 (SW)
- new net: R100.1, U10.10 (RON)
- new net: C80.1, U10.11 (VCC)
- new net: C45.2, U10.3 (BOOT)
- new net: R95.2, U10.5 (VOUT)
- new net: R105.2, U10.6 (CS)
- new net: R150.1, U10.8 (DIM)
- new net: C79.1, U10.9 (COMP)
- new net: C69.1, C70.1, D30.2 (A), J15.1 (Pin_1), L10.2, R95.1
- new net: C69.2, C70.2, J15.2 (Pin_2), R105.1, R151.2, R152.2, R153.2, R154.2, R155.2, R156.2, R157.2, R158.2, R159.2, R160.2, R170.1
- new net: D40.3 (+), R170.2
- new net: D40.4 (-), R175.2, R180.1
- new net: C85.1, D45.1 (K), L15.1, U15.1 (SW), U15.2 (SW)
- new net: R190.1, U15.10 (RON)
- new net: C120.1, U15.11 (VCC)
- new net: C85.2, U15.3 (BOOT)
- new net: R185.2, U15.5 (VOUT)
- new net: R195.2, U15.6 (CS)
- new net: R240.1, U15.8 (DIM)
- new net: C119.1, U15.9 (COMP)
- new net: C109.1, C110.1, D50.2 (A), J20.1 (Pin_1), L15.2, R185.1
- new net: C109.2, C110.2, J20.2 (Pin_2), R195.1, R241.2, R242.2, R243.2, R244.2, R245.2, R246.2, R247.2, R248.2, R249.2, R250.2, R260.1
- new net: D60.3 (+), R260.2
- new net: D60.4 (-), R265.2, R270.1
- new net: C125.1, D65.1 (K), L20.1, U20.1 (SW), U20.2 (SW)
- new net: R280.1, U20.10 (RON)
- new net: C160.1, U20.11 (VCC)
- new net: C125.2, U20.3 (BOOT)
- new net: R275.2, U20.5 (VOUT)
- new net: R285.2, U20.6 (CS)
- new net: R330.1, U20.8 (DIM)
- new net: C159.1, U20.9 (COMP)
- new net: C149.1, C150.1, D70.2 (A), J25.1 (Pin_1), L20.2, R275.1
- new net: C149.2, C150.2, J25.2 (Pin_2), R285.1, R331.2, R332.2, R333.2, R334.2, R335.2, R336.2, R337.2, R338.2, R339.2, R340.2, R350.1
- new net: D80.3 (+), R350.2
- new net: D80.4 (-), R355.2, R360.1
- new net: C165.1, D85.1 (K), L25.1, U25.1 (SW), U25.2 (SW)
- new net: R370.1, U25.10 (RON)
- new net: C200.1, U25.11 (VCC)
- new net: C165.2, U25.3 (BOOT)
- new net: R365.2, U25.5 (VOUT)
- new net: R375.2, U25.6 (CS)
- new net: R420.1, U25.8 (DIM)
- new net: C199.1, U25.9 (COMP)
- new net: C189.1, C190.1, D90.2 (A), J30.1 (Pin_1), L25.2, R365.1
- new net: C189.2, C190.2, J30.2 (Pin_2), R375.1, R421.2, R422.2, R423.2, R424.2, R425.2, R426.2, R427.2, R428.2, R429.2, R430.2, R440.1
- new net: D100.3 (+), R440.2
- new net: D100.4 (-), R445.2, R450.1
- new net: R456.1, R457.2
- new net +5v_IN_ISO: C218.1, C222.1, C223.1, J32.4, J33.4, R460.2, U30.3 (VDD), U34.8 (VCC), U35.10 (EN2), U35.16 (VCC2)
- new net A_ISO: J32.2, J33.2, R459.1, R463.2
- new net B_ISO: J32.1, J33.1, R461.2, SW1.2
- new net DE_ISO: R464.2, U34.2 (~RE), U34.3 (DE), U35.13 (OUTB)
- new net GND_5v_IN_ISO: C218.2, C222.2, C223.2, D104.3, J32.3, J32.SH, J33.3, J33.SH, R458.1, R464.1, U30.2 (VSS), U34.5 (GND), U35.15 (GND2), U35.9 (GND2)
- new net IN_+24v: C221.1, D105.1 (+), J32.7, J33.7, U36.1 (VIN)
- new net IN_GND_24v: C219.2, C221.2, D101.2 (-VIN), D102.2 (A), D105.3 (-), J32.8, J33.8, R465.1, U36.3 (GND), U36.5 (~ON~/OFF)
- new net LED_S1: R468.1, U37.3 (QD)
- new net LED_S2: R467.1, U37.2 (QC)
- new net LED_S3: R466.1, U37.1 (QB)
- new net OFF_CH1: D11.1 (G), R71.2, U26.15 (QA)
- new net OFF_CH10: D92.1 (G), R432.2, U27.1 (QB)
- new net OFF_CH11: D13.1 (G), R73.2, U27.2 (QC)
- new net OFF_CH12: D33.1 (G), R163.2, U27.3 (QD)
- new net OFF_CH13: D53.1 (G), R253.2, U27.4 (QE)
- new net OFF_CH14: D73.1 (G), R343.2, U27.5 (QF)
- new net OFF_CH15: D93.1 (G), R433.2, U27.6 (QG)
- new net OFF_CH16: D14.1 (G), R74.2, U27.7 (QH)
- new net OFF_CH17: D34.1 (G), R164.2, U32.15 (QA)
- new net OFF_CH18: D54.1 (G), R254.2, U32.1 (QB)
- new net OFF_CH19: D74.1 (G), R344.2, U32.2 (QC)
- new net OFF_CH2: D31.1 (G), R161.2, U26.1 (QB)
- new net OFF_CH20: D94.1 (G), R434.2, U32.3 (QD)
- new net OFF_CH21: D15.1 (G), R75.2, U32.4 (QE)
- new net OFF_CH22: D35.1 (G), R165.2, U32.5 (QF)
- new net OFF_CH23: D55.1 (G), R255.2, U32.6 (QG)
- new net OFF_CH24: D75.1 (G), R345.2, U32.7 (QH)
- new net OFF_CH25: D95.1 (G), R435.2, U37.15 (QA)
- new net OFF_CH3: D51.1 (G), R251.2, U26.2 (QC)
- new net OFF_CH4: D71.1 (G), R341.2, U26.3 (QD)
- new net OFF_CH5: D91.1 (G), R431.2, U26.4 (QE)
- new net OFF_CH6: D12.1 (G), R72.2, U26.5 (QF)
- new net OFF_CH7: D32.1 (G), R162.2, U26.6 (QG)
- new net OFF_CH8: D52.1 (G), R252.2, U26.7 (QH)
- new net OFF_CH9: D72.1 (G), R342.2, U27.15 (QA)
- new net RX: JP2.2 (B), JP4.1 (A), U35.6 (OUTD)
- new net RX_ISO: R460.1, U30.4 (RXD), U34.1 (RO), U35.11 (IND)
- new net TX: JP1.2 (B), JP3.1 (A), U35.5 (INC)
- new net TX_ISO: U30.1 (TXD), U34.4 (DI), U35.12 (OUTC)
- no-connect marks 0 -> 13
Other:
- note added: "Изолированная часть. Приемо передатчик RS-485/CAN"
- moved on the sheet: U29

Commit message: Плата
исправил ошибку в схеме (выключение канала). Разместил детали для одного канала (ушло времен 1 час)
Parts:
- U1, U10, U11, U12, U13, U14, U15, U16, U17, U18, U19, U2, U20, U21, U22, U23, U24, U25, U3, U4, U5, U6, U7, U8, U9: symbol Regulator_Switching:LM3406 -> LED_driver-rescue:LM3406-Regulator_Switching
- U26, U27, U32, U37: symbol 74xx:74HC595 -> LED_driver-rescue:74HC595-74xx
- U33: symbol Memory_Flash:GD25Q16C -> LED_driver-rescue:GD25Q16C-Memory_Flash
Connections:
- net at R9.1, U4.10 (RON): now also D14.3 (D)
- net at C135.1, C136.1, C137.1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: no longer D14.3 (D), D34.3 (D), D54.3 (D), D74.3 (D), D94.3 (D)
- net at R99.1, U9.10 (RON): now also D34.3 (D)
- net at R189.1, U14.10 (RON): now also D54.3 (D)
- net at R279.1, U19.10 (RON): now also D74.3 (D)
- net at R369.1, U24.10 (RON): now also D94.3 (D)
- net at R8.1, U3.10 (RON): now also D13.3 (D)
- net at C12.1, C13.1, C132.1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: no longer D13.3 (D), D33.3 (D), D53.3 (D), D73.3 (D), D93.3 (D)
- net at R98.1, U8.10 (RON): now also D33.3 (D)
- net at R188.1, U13.10 (RON): now also D53.3 (D)
- net at R278.1, U18.10 (RON): now also D73.3 (D)
- net at R368.1, U23.10 (RON): now also D93.3 (D)
- net at R7.1, U2.10 (RON): now also D12.3 (D)
- net at C10.1, C11.1, C129.1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: no longer D12.3 (D), D32.3 (D), D52.3 (D), D72.3 (D), D92.3 (D)
- net at R97.1, U7.10 (RON): now also D32.3 (D)
- net at R187.1, U12.10 (RON): now also D52.3 (D)
- net at R277.1, U17.10 (RON): now also D72.3 (D)
- net at R367.1, U22.10 (RON): now also D92.3 (D)
- net at R6.1, U1.10 (RON): now also D11.3 (D)
- net at C126.1, C127.1, C128.1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: no longer D11.3 (D), D31.3 (D), D51.3 (D), D71.3 (D), D91.3 (D)
- net at R96.1, U6.10 (RON): now also D31.3 (D)
- net at R186.1, U11.10 (RON): now also D51.3 (D)
- net at R276.1, U16.10 (RON): now also D71.3 (D)
- net at R366.1, U21.10 (RON): now also D91.3 (D)
- net at R10.1, U5.10 (RON): now also D15.3 (D)
- net at C100.1, C138.1, C139.1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: no longer D15.3 (D), D35.3 (D), D55.3 (D), D75.3 (D), D95.3 (D)
- net at R100.1, U10.10 (RON): now also D35.3 (D)
- net at R190.1, U15.10 (RON): now also D55.3 (D)
- net at R280.1, U20.10 (RON): now also D75.3 (D)
- net at R370.1, U25.10 (RON): now also D95.3 (D)
