File: schem/LED_driver/LED_driver.sch (KiCad schematic (older format))
At the start: 922 parts, among them J1 Screw_Terminal_01x04, J10 Screw_Terminal_01x02, J11 Screw_Terminal_01x02, J12 Screw_Terminal_01x02, J13 Screw_Terminal_01x02, J14 Screw_Terminal_01x02, J15 Screw_Terminal_01x02, J16 Screw_Terminal_01x02, J17 Screw_Terminal_01x02, J18 Screw_Terminal_01x02, J19 Screw_Terminal_01x02, J2 Screw_Terminal_01x04, J20 Screw_Terminal_01x02, J21 Screw_Terminal_01x02, J22 Screw_Terminal_01x02, J23 Screw_Terminal_01x02, J24 Screw_Terminal_01x02, J25 Screw_Terminal_01x02, J26 Screw_Terminal_01x02, J27 Screw_Terminal_01x02, J28 Screw_Terminal_01x02, J29 Screw_Terminal_01x02, J3 Screw_Terminal_01x04, J30 Screw_Terminal_01x02, J31 SWD, J32 RJ45_Shielded, J33 RJ45_Shielded, J34 DEBUG, J35 Screw_Terminal_01x02, J4 Screw_Terminal_01x04, J5 Screw_Terminal_01x04, J6 Screw_Terminal_01x02, J7 Screw_Terminal_01x02, J8 Screw_Terminal_01x02, J9 Screw_Terminal_01x02, SW1 SW_DIP_x01, U1 LM3406, U10 LM3406, U11 LM3406, U12 LM3406, U13 LM3406, U14 LM3406, U15 LM3406, U16 LM3406, U17 LM3406, U18 LM3406, U19 LM3406, U2 LM3406, U20 LM3406, U21 LM3406, U22 LM3406, U23 LM3406, U24 LM3406, U25 LM3406, U26 74HC595, U27 74HC595, U28 TL431LP, U29 STM32F303VCTx, U3 LM3406, U30 MCP2551-I_SN, U31 LM1117-3.3, U32 74HC595, U33 GD25Q16C, U34 MAX3485, U35 ISO7341C, U36 LM2596S-ADJ, U37 74HC595, U4 LM3406, U5 LM3406, U6 LM3406, U7 LM3406, U8 LM3406, U9 LM3406, Y1 Crystal_Small

Commit message: PCB
Parts:
- removed J1, J2, J3, J4, J5: Screw_Terminal_01x04, TerminalBlock:TerminalBlock_bornier-4_P5.08mm, symbol Connector:Screw_Terminal_01x04
- added J1, J2, J3, J4, J5: Screw_Terminal_01x02, TerminalBlock:TerminalBlock_bornier-2_P5.08mm, symbol Connector:Screw_Terminal_01x02
Connections:
- net GND: now also J1.1 (Pin_1), J2.1 (Pin_1), J3.1 (Pin_1), J4.1 (Pin_1), J5.1 (Pin_1)
- net at C135.1, C136.1, C137.1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: now also J4.2 (Pin_2)
- net at C12.1, C13.1, C132.1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: now also J3.2 (Pin_2)
- net at C10.1, C11.1, C129.1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: now also J2.2 (Pin_2)
- net at C126.1, C127.1, C128.1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: now also J1.2 (Pin_2)
- net at C100.1, C138.1, C139.1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: now also J5.2 (Pin_2)
Changed lines of the file:
@@
 $EndComp
 $Comp
-L Connector:Screw_Terminal_01x04 J5
-U 1 1 61347956
-P 38950 2150
-F 0 "J5" V 38914 1862 50  0000 R CNN
-F 1 "Screw_Terminal_01x04" V 38823 1862 50  0000 R CNN
-F 2 "TerminalBlock:TerminalBlock_bornier-4_P5.08mm" H 38950 2150 50  0001 C CNN
-F 3 "~" H 38950 2150 50  0001 C CNN
-	1    38950 2150
-	0    -1   -1   0
-$EndComp
-$Comp
 L Connector:Screw_Terminal_01x02 J10
 U 1 1 6134795C
@@
 Wire Wire Line
 	39150 2350 39150 2700
-Connection ~ 39150 2350
 Wire Wire Line
 	38950 2350 38850 2350
-Connection ~ 38850 2350
 Wire Wire Line
 	39650 3400 39150 3400
@@
 $EndComp
 $Comp
-L Connector:Screw_Terminal_01x04 J4
-U 1 1 5F2AF11E
-P 30550 2150
-F 0 "J4" V 30514 1862 50  0000 R CNN
-F 1 "Screw_Terminal_01x04" V 30423 1862 50  0000 R CNN
-F 2 "TerminalBlock:TerminalBlock_bornier-4_P5.08mm" H 30550 2150 50  0001 C CNN
-F 3 "~" H 30550 2150 50  0001 C CNN
-	1    30550 2150
-	0    -1   -1   0
-$EndComp
-$Comp
 L Connector:Screw_Terminal_01x02 J9
 U 1 1 5F2AF124
@@
 Wire Wire Line
 	30750 2350 30750 2600
-Connection ~ 30750 2350
 Wire Wire Line
 	30550 2350 30450 2350
-Connection ~ 30450 2350
 Wire Wire Line
 	31250 3400 30750 3400
@@
 $EndComp
 $Comp
-L Connector:Screw_Terminal_01x04 J3
-U 1 1 5F4D4BA6
-P 22200 2150
-F 0 "J3" V 22164 1862 50  0000 R CNN
-F 1 "Screw_Terminal_01x04" V 22073 1862 50  0000 R CNN
-F 2 "TerminalBlock:TerminalBlock_bornier-4_P5.08mm" H 22200 2150 50  0001 C CNN
-F 3 "~" H 22200 2150 50  0001 C CNN
-	1    22200 2150
-	0    -1   -1   0
-$EndComp
-$Comp
 L Connector:Screw_Terminal_01x02 J8
 U 1 1 5F4D4BAC
@@
 Wire Wire Line
 	22400 2350 22400 2600
-Connection ~ 22400 2350
 Wire Wire Line
 	22200 2350 22100 2350
-Connection ~ 22100 2350
 Wire Wire Line
 	22900 3400 22400 3400
@@
 $EndComp
 $Comp
-L Connector:Screw_Terminal_01x04 J2
-U 1 1 5FD0C18C
-P 13750 2150
-F 0 "J2" V 13714 1862 50  0000 R CNN
-F 1 "Screw_Terminal_01x04" V 13623 1862 50  0000 R CNN
-F 2 "TerminalBlock:TerminalBlock_bornier-4_P5.08mm" H 13750 2150 50  0001 C CNN
-F 3 "~" H 13750 2150 50  0001 C CNN
-	1    13750 2150
-	0    -1   -1   0
-$EndComp
-$Comp
 L Connector:Screw_Terminal_01x02 J7
 U 1 1 5FD0C192
@@
 Wire Wire Line
 	13950 2350 13950 2600
-Connection ~ 13950 2350
 Wire Wire Line
 	13750 2350 13650 2350
-Connection ~ 13650 2350
 Wire Wire Line
 	14450 3400 13950 3400
@@
 $EndComp
 $Comp
-L Connector:Screw_Terminal_01x04 J1
-U 1 1 604301A2
-P 5450 2150
-F 0 "J1" V 5414 1862 50  0000 R CNN
-F 1 "Screw_Terminal_01x04" V 5323 1862 50  0000 R CNN
-F 2 "TerminalBlock:TerminalBlock_bornier-4_P5.08mm" H 5450 2150 50  0001 C CNN
-F 3 "~" H 5450 2150 50  0001 C CNN
-	1    5450 2150
-	0    -1   -1   0
-$EndComp
-$Comp
 L Connector:Screw_Terminal_01x02 J6
 U 1 1 604301A8
@@
 Wire Wire Line
 	5650 2350 5650 2650
-Connection ~ 5650 2350
 Wire Wire Line
 	5450 2350 5350 2350
-Connection ~ 5350 2350
 Wire Wire Line
 	6150 3400 5650 3400
@@
 Wire Wire Line
 	41750 3650 41050 3650
+Connection ~ 41750 3750
+Wire Wire Line
+	41750 3750 41700 3750
+Wire Wire Line
+	41050 3650 41050 4200
+$Comp
+L Connector:Screw_Terminal_01x02 J1
+U 1 1 6024577D
+P 5450 2150
+F 0 "J1" H 5530 2142 50  0000 L CNN
+F 1 "Screw_Terminal_01x02" H 5530 2051 50  0000 L CNN
+F 2 "TerminalBlock:TerminalBlock_bornier-2_P5.08mm" H 5450 2150 50  0001 C CNN
+F 3 "~" H 5450 2150 50  0001 C CNN
+	1    5450 2150
+	0    -1   -1   0
+$EndComp
+$Comp
+L Connector:Screw_Terminal_01x02 J2
+U 1 1 6024AF0C
+P 13750 2150
+F 0 "J2" H 13830 2142 50  0000 L CNN
+F 1 "Screw_Terminal_01x02" H 13830 2051 50  0000 L CNN
+F 2 "TerminalBlock:TerminalBlock_bornier-2_P5.08mm" H 13750 2150 50  0001 C CNN
+F 3 "~" H 13750 2150 50  0001 C CNN
+	1    13750 2150
+	0    -1   -1   0
+$EndComp
+$Comp
+L Connector:Screw_Terminal_01x02 J3
+U 1 1 6025D0D5
+P 22200 2150
+F 0 "J3" H 22280 2142 50  0000 L CNN
+F 1 "Screw_Terminal_01x02" H 22280 2051 50  0000 L CNN
+F 2 "TerminalBlock:TerminalBlock_bornier-2_P5.08mm" H 22200 2150 50  0001 C CNN
+F 3 "~" H 22200 2150 50  0001 C CNN
+	1    22200 2150
+	0    -1   -1   0
+$EndComp
+$Comp
+L Connector:Screw_Terminal_01x02 J4
+U 1 1 60267804
+P 30550 2150
+F 0 "J4" H 30630 2142 50  0000 L CNN
+F 1 "Screw_Terminal_01x02" H 30630 2051 50  0000 L CNN
+F 2 "TerminalBlock:TerminalBlock_bornier-2_P5.08mm" H 30550 2150 50  0001 C CNN
+F 3 "~" H 30550 2150 50  0001 C CNN
+	1    30550 2150
+	0    -1   -1   0
+$EndComp
+$Comp
+L Connector:Screw_Terminal_01x02 J5
+U 1 1 60272DD0
+P 38950 2150
+F 0 "J5" H 39030 2142 50  0000 L CNN
+F 1 "Screw_Terminal_01x02" H 39030 2051 50  0000 L CNN
+F 2 "TerminalBlock:TerminalBlock_bornier-2_P5.08mm" H 38950 2150 50  0001 C CNN
+F 3 "~" H 38950 2150 50  0001 C CNN
+	1    38950 2150
+	0    -1   -1   0
+$EndComp
 Wire Wire Line
 	23800 26300 24600 26300
@@
 Wire Bus Line
 	21300 26250 21300 31200
-Connection ~ 41750 3750
-Wire Wire Line
-	41750 3750 41700 3750
-Wire Wire Line
-	41050 3650 41050 4200
 $EndSCHEMATC
