File: schem/LED_driver/LED_driver.sch (KiCad schematic (older format))
At the start: 922 parts, among them J1 Screw_Terminal_01x02, J10 Screw_Terminal_01x02, J11 Screw_Terminal_01x02, J12 Screw_Terminal_01x02, J13 Screw_Terminal_01x02, J14 Screw_Terminal_01x02, J15 Screw_Terminal_01x02, J16 Screw_Terminal_01x02, J17 Screw_Terminal_01x02, J18 Screw_Terminal_01x02, J19 Screw_Terminal_01x02, J2 Screw_Terminal_01x02, J20 Screw_Terminal_01x02, J21 Screw_Terminal_01x02, J22 Screw_Terminal_01x02, J23 Screw_Terminal_01x02, J24 Screw_Terminal_01x02, J25 Screw_Terminal_01x02, J26 Screw_Terminal_01x02, J27 Screw_Terminal_01x02, J28 Screw_Terminal_01x02, J29 Screw_Terminal_01x02, J3 Screw_Terminal_01x02, J30 Screw_Terminal_01x02, J31 SWD, J32 RJ45_Shielded, J33 RJ45_Shielded, J34 DEBUG, J35 Screw_Terminal_01x02, J4 Screw_Terminal_01x02, J5 Screw_Terminal_01x02, J6 Screw_Terminal_01x02, J7 Screw_Terminal_01x02, J8 Screw_Terminal_01x02, J9 Screw_Terminal_01x02, SW1 SW_DIP_x01, U1 LM3406, U10 LM3406, U11 LM3406, U12 LM3406, U13 LM3406, U14 LM3406, U15 LM3406, U16 LM3406, U17 LM3406, U18 LM3406, U19 LM3406, U2 LM3406, U20 LM3406, U21 LM3406, U22 LM3406, U23 LM3406, U24 LM3406, U25 LM3406, U26 74HC595, U27 74HC595, U28 TL431LP, U29 STM32F303VCTx, U3 LM3406, U30 MCP2551-I_SN, U31 LM1117-3.3, U32 74HC595, U33 GD25Q16C, U34 MAX3485, U35 ISO7341C, U36 LM2596S-ADJ, U37 74HC595, U4 LM3406, U5 LM3406, U6 LM3406, U7 LM3406, U8 LM3406, U9 LM3406, Y1 Crystal_Small

Commit message: Плата
Плата закончена
Parts:
- added D107: D_Schottky, Diode_SMD:D_SMC, symbol Device:D_Schottky
- added R470: nc, Resistor_SMD:R_0805_2012Metric, symbol Device:R
- added TP19, TP20: TestPoint, TestPoint:TestPoint_Plated_Hole_D4.0mm, symbol Connector:TestPoint
- TP16: value C13 -> TestPoint; footprint TestPoint:TestPoint_Pad_D1.0mm -> TestPoint:TestPoint_Plated_Hole_D4.0mm
- TP17: value C14 -> TestPoint; footprint TestPoint:TestPoint_Pad_D1.0mm -> TestPoint:TestPoint_Plated_Hole_D4.0mm
- TP18: value C15 -> TestPoint; footprint TestPoint:TestPoint_Pad_D1.0mm -> TestPoint:TestPoint_Plated_Hole_D4.0mm
- TP8: value E6 -> TestPoint; footprint TestPoint:TestPoint_Pad_D1.0mm -> TestPoint:TestPoint_Plated_Hole_D4.0mm
Connections:
- net IN_+24v: now also D107.2 (A); no longer C221.1, D105.1 (+), U36.1 (VIN)
- net at U29.5 (PE6): no longer TP8.1
- net at U29.7 (PC13): no longer TP16.1
- net at U29.8 (PC14): no longer TP17.1
- net at U29.9 (PC15): no longer TP18.1
- net at R462.1, R465.2, U36.4 (FB): now also R470.2
- new net: C221.1, D105.1 (+), D107.1 (K), R470.1, U36.1 (VIN)
- no-connect marks 13 -> 23
Changed lines of the file:
@@
 	11000 30250 11300 30250
 Wire Wire Line
-	10900 30050 11200 30050
+	10900 30050 10950 30050
 Wire Wire Line
 	11200 30050 11200 30150
@@
 Text Label 10400 30650 2    50   ~ 0
 IN_GND_24v
-Text Label 9700 29950 2    50   ~ 0
+Text Label 10025 29450 0    50   ~ 0
 IN_+24v
-Wire Wire Line
-	9700 29950 9700 30050
 $Comp
 L Device:CP_Small C219
@@
 	23800 29100 24550 29100
 $Comp
-L Connector:TestPoint TP16
-U 1 1 66F2DB7A
-P 23800 29900
-F 0 "TP16" V 23754 30088 50  0000 L CNN
-F 1 "C13" V 23845 30088 50  0000 L CNN
-F 2 "TestPoint:TestPoint_Pad_D1.0mm" H 24000 29900 50  0001 C CNN
-F 3 "~" H 24000 29900 50  0001 C CNN
-	1    23800 29900
-	0    1    1    0
-$EndComp
-$Comp
-L Connector:TestPoint TP18
-U 1 1 66F2FF71
-P 23800 30100
-F 0 "TP18" V 23754 30288 50  0000 L CNN
-F 1 "C15" V 23845 30288 50  0000 L CNN
-F 2 "TestPoint:TestPoint_Pad_D1.0mm" H 24000 30100 50  0001 C CNN
-F 3 "~" H 24000 30100 50  0001 C CNN
-	1    23800 30100
-	0    1    1    0
-$EndComp
-$Comp
-L Connector:TestPoint TP17
-U 1 1 66F30535
-P 24600 30000
-F 0 "TP17" V 24554 30188 50  0000 L CNN
-F 1 "C14" V 24645 30188 50  0000 L CNN
-F 2 "TestPoint:TestPoint_Pad_D1.0mm" H 24800 30000 50  0001 C CNN
-F 3 "~" H 24800 30000 50  0001 C CNN
-	1    24600 30000
-	0    1    1    0
-$EndComp
-Wire Wire Line
-	23800 30000 24600 30000
-$Comp
 L Connector:TestPoint TP11
 U 1 1 67D38C03
@@
 	21750 27900 22200 27900
 $Comp
-L Connector:TestPoint TP8
-U 1 1 68B430F6
-P 21850 27500
-F 0 "TP8" V 21804 27688 50  0000 L CNN
-F 1 "E6" V 21895 27688 50  0000 L CNN
-F 2 "TestPoint:TestPoint_Pad_D1.0mm" H 22050 27500 50  0001 C CNN
-F 3 "~" H 22050 27500 50  0001 C CNN
-	1    21850 27500
-	0    -1   -1   0
-$EndComp
-$Comp
 L Connector:TestPoint TP10
 U 1 1 68B43920
@@
 $EndComp
 Wire Wire Line
-	22200 27500 21850 27500
-Wire Wire Line
 	22200 27600 21250 27600
 $Comp
@@
 	1    0    0    1
 $EndComp
+Text Label 22150 28300 2    50   ~ 0
+Isens_CH14
+Text Label 23850 28100 0    50   ~ 0
+Isens_CH16
+$Comp
+L Device:D_Schottky D107
+U 1 1 60896D1B
+P 9875 29450
+F 0 "D107" H 9875 29234 50  0000 C CNN
+F 1 "D_Schottky" H 9875 29325 50  0000 C CNN
+F 2 "Diode_SMD:D_SMC" V 9966 29529 60  0001 L CNN
+F 3 "" H 9875 29450 60  0000 C CNN
+	1    9875 29450
+	1    0    0    -1
+$EndComp
+Wire Wire Line
+	9700 29450 9725 29450
+$Comp
+L Device:R R470
+U 1 1 602F6DE7
+P 10400 29600
+F 0 "R470" V 10500 29600 50  0000 C CNN
+F 1 "nc" V 10400 29600 50  0000 C CNN
+F 2 "Resistor_SMD:R_0805_2012Metric" H 10470 29509 30  0001 L CNN
+F 3 "" H 10400 29600 30  0000 C CNN
+	1    10400 29600
+	0    -1   1    0
+$EndComp
+Wire Wire Line
+	10250 29600 9700 29600
+Wire Wire Line
+	9700 29450 9700 29600
+Connection ~ 9700 29600
+Wire Wire Line
+	9700 29600 9700 30050
+Wire Wire Line
+	10550 29600 10950 29600
+Wire Wire Line
+	10950 29600 10950 30050
+Connection ~ 10950 30050
+Wire Wire Line
+	10950 30050 11200 30050
+NoConn ~ 22200 27500
+NoConn ~ 23800 29900
+NoConn ~ 23800 30000
+NoConn ~ 23800 30100
+$Comp
+L Connector:TestPoint TP8
+U 1 1 66DB9EE4
+P 33075 27875
+F 0 "TP8" H 33133 28038 50  0000 L CNN
+F 1 "TestPoint" H 33133 27947 50  0000 L CNN
+F 2 "TestPoint:TestPoint_Plated_Hole_D4.0mm" H 33133 27856 50  0000 L CNN
+F 3 "~" H 33275 27875 50  0001 C CNN
+	1    33075 27875
+	1    0    0    -1
+$EndComp
+NoConn ~ 33075 27875
+$Comp
+L Connector:TestPoint TP16
+U 1 1 67C5012B
+P 33075 28100
+F 0 "TP16" H 33133 28263 50  0000 L CNN
+F 1 "TestPoint" H 33133 28172 50  0000 L CNN
+F 2 "TestPoint:TestPoint_Plated_Hole_D4.0mm" H 33133 28081 50  0000 L CNN
+F 3 "~" H 33275 28100 50  0001 C CNN
+	1    33075 28100
+	1    0    0    -1
+$EndComp
+NoConn ~ 33075 28100
+$Comp
+L Connector:TestPoint TP17
+U 1 1 68ADA86E
+P 33075 28350
+F 0 "TP17" H 33133 28513 50  0000 L CNN
+F 1 "TestPoint" H 33133 28422 50  0000 L CNN
+F 2 "TestPoint:TestPoint_Plated_Hole_D4.0mm" H 33133 28331 50  0000 L CNN
+F 3 "~" H 33275 28350 50  0001 C CNN
+	1    33075 28350
+	1    0    0    -1
+$EndComp
+NoConn ~ 33075 28350
+$Comp
+L Connector:TestPoint TP18
+U 1 1 69964F33
+P 33075 28625
+F 0 "TP18" H 33133 28788 50  0000 L CNN
+F 1 "TestPoint" H 33133 28697 50  0000 L CNN
+F 2 "TestPoint:TestPoint_Plated_Hole_D4.0mm" H 33133 28606 50  0000 L CNN
+F 3 "~" H 33275 28625 50  0001 C CNN
+	1    33075 28625
+	1    0    0    -1
+$EndComp
+NoConn ~ 33075 28625
+$Comp
+L Connector:TestPoint TP19
+U 1 1 6A7EF4EC
+P 33075 28875
+F 0 "TP19" H 33133 29038 50  0000 L CNN
+F 1 "TestPoint" H 33133 28947 50  0000 L CNN
+F 2 "TestPoint:TestPoint_Plated_Hole_D4.0mm" H 33133 28856 50  0000 L CNN
+F 3 "~" H 33275 28875 50  0001 C CNN
+	1    33075 28875
+	1    0    0    -1
+$EndComp
+NoConn ~ 33075 28875
+$Comp
+L Connector:TestPoint TP20
+U 1 1 6B679B93
+P 33075 29150
+F 0 "TP20" H 33133 29313 50  0000 L CNN
+F 1 "TestPoint" H 33133 29222 50  0000 L CNN
+F 2 "TestPoint:TestPoint_Plated_Hole_D4.0mm" H 33133 29131 50  0000 L CNN
+F 3 "~" H 33275 29150 50  0001 C CNN
+	1    33075 29150
+	1    0    0    -1
+$EndComp
+NoConn ~ 33075 29150
 Wire Wire Line
 	23800 26300 24600 26300
@@
 Wire Bus Line
 	21300 26250 21300 31200
-Text Label 22150 28300 2    50   ~ 0
-Isens_CH14
-Text Label 23850 28100 0    50   ~ 0
-Isens_CH16
 $EndSCHEMATC

Commit message: Programming
проект переведен в C++. Добавлен класс flash, проверен hc595
Parts:
- R161, R162, R163, R164, R165, R251, R252, R253, R254, R255, R341, R342, R343, R344, R345, R431, R432, R433, R434, R435, R71, R72, R73, R74, R75: value 100K -> 10k
- R466: value 1.5k -> 10k
- R467: value 1k -> 10k; footprint Resistor_SMD:R_0805_2012Metric_Pad1.15x1.40mm_HandSolder -> Resistor_SMD:R_0805_2012Metric
- R468: value 750 Om -> 10k
Changed lines of the file:
@@
 P 40800 4650
 F 0 "R75" V 40700 4650 50  0000 C CNN
-F 1 "100K" V 40800 4650 50  0000 C CNN
+F 1 "10k" V 40800 4650 50  0000 C CNN
 F 2 "Resistor_SMD:R_0805_2012Metric" H 40870 4559 30  0001 L CNN
 F 3 "" H 40800 4650 30  0000 C CNN
@@
 P 40800 8700
 F 0 "R165" V 40700 8700 50  0000 C CNN
-F 1 "100K" V 40800 8700 50  0000 C CNN
+F 1 "10k" V 40800 8700 50  0000 C CNN
 F 2 "Resistor_SMD:R_0805_2012Metric" H 40870 8609 30  0001 L CNN
 F 3 "" H 40800 8700 30  0000 C CNN
@@
 P 40800 12750
 F 0 "R255" V 40700 12750 50  0000 C CNN
-F 1 "100K" V 40800 12750 50  0000 C CNN
+F 1 "10k" V 40800 12750 50  0000 C CNN
 F 2 "Resistor_SMD:R_0805_2012Metric" H 40870 12659 30  0001 L CNN
 F 3 "" H 40800 12750 30  0000 C CNN
@@
 P 40800 16800
 F 0 "R345" V 40700 16800 50  0000 C CNN
-F 1 "100K" V 40800 16800 50  0000 C CNN
+F 1 "10k" V 40800 16800 50  0000 C CNN
 F 2 "Resistor_SMD:R_0805_2012Metric" H 40870 16709 30  0001 L CNN
 F 3 "" H 40800 16800 30  0000 C CNN
@@
 P 40800 20850
 F 0 "R435" V 40700 20850 50  0000 C CNN
-F 1 "100K" V 40800 20850 50  0000 C CNN
+F 1 "10k" V 40800 20850 50  0000 C CNN
 F 2 "Resistor_SMD:R_0805_2012Metric" H 40870 20759 30  0001 L CNN
 F 3 "" H 40800 20850 30  0000 C CNN
@@
 P 32400 4650
 F 0 "R74" V 32300 4650 50  0000 C CNN
-F 1 "100K" V 32400 4650 50  0000 C CNN
+F 1 "10k" V 32400 4650 50  0000 C CNN
 F 2 "Resistor_SMD:R_0805_2012Metric" H 32470 4559 30  0001 L CNN
 F 3 "" H 32400 4650 30  0000 C CNN
@@
 P 32400 8700
 F 0 "R164" V 32300 8700 50  0000 C CNN
-F 1 "100K" V 32400 8700 50  0000 C CNN
+F 1 "10k" V 32400 8700 50  0000 C CNN
 F 2 "Resistor_SMD:R_0805_2012Metric" H 32470 8609 30  0001 L CNN
 F 3 "" H 32400 8700 30  0000 C CNN
@@
 P 32400 12750
 F 0 "R254" V 32300 12750 50  0000 C CNN
-F 1 "100K" V 32400 12750 50  0000 C CNN
+F 1 "10k" V 32400 12750 50  0000 C CNN
 F 2 "Resistor_SMD:R_0805_2012Metric" H 32470 12659 30  0001 L CNN
 F 3 "" H 32400 12750 30  0000 C CNN
@@
 P 32400 16800
 F 0 "R344" V 32300 16800 50  0000 C CNN
-F 1 "100K" V 32400 16800 50  0000 C CNN
+F 1 "10k" V 32400 16800 50  0000 C CNN
 F 2 "Resistor_SMD:R_0805_2012Metric" H 32470 16709 30  0001 L CNN
 F 3 "" H 32400 16800 30  0000 C CNN
@@
 P 32400 20850
 F 0 "R434" V 32300 20850 50  0000 C CNN
-F 1 "100K" V 32400 20850 50  0000 C CNN
+F 1 "10k" V 32400 20850 50  0000 C CNN
 F 2 "Resistor_SMD:R_0805_2012Metric" H 32470 20759 30  0001 L CNN
 F 3 "" H 32400 20850 30  0000 C CNN
@@
 P 24050 4650
 F 0 "R73" V 23950 4650 50  0000 C CNN
-F 1 "100K" V 24050 4650 50  0000 C CNN
+F 1 "10k" V 24050 4650 50  0000 C CNN
 F 2 "Resistor_SMD:R_0805_2012Metric" H 24120 4559 30  0001 L CNN
 F 3 "" H 24050 4650 30  0000 C CNN
@@
 P 24050 8700
 F 0 "R163" V 23950 8700 50  0000 C CNN
-F 1 "100K" V 24050 8700 50  0000 C CNN
+F 1 "10k" V 24050 8700 50  0000 C CNN
 F 2 "Resistor_SMD:R_0805_2012Metric" H 24120 8609 30  0001 L CNN
 F 3 "" H 24050 8700 30  0000 C CNN
@@
 P 24050 12750
 F 0 "R253" V 23950 12750 50  0000 C CNN
-F 1 "100K" V 24050 12750 50  0000 C CNN
+F 1 "10k" V 24050 12750 50  0000 C CNN
 F 2 "Resistor_SMD:R_0805_2012Metric" H 24120 12659 30  0001 L CNN
 F 3 "" H 24050 12750 30  0000 C CNN
@@
 P 24050 16800
 F 0 "R343" V 23950 16800 50  0000 C CNN
-F 1 "100K" V 24050 16800 50  0000 C CNN
+F 1 "10k" V 24050 16800 50  0000 C CNN
 F 2 "Resistor_SMD:R_0805_2012Metric" H 24120 16709 30  0001 L CNN
 F 3 "" H 24050 16800 30  0000 C CNN
@@
 P 24050 20850
 F 0 "R433" V 23950 20850 50  0000 C CNN
-F 1 "100K" V 24050 20850 50  0000 C CNN
+F 1 "10k" V 24050 20850 50  0000 C CNN
 F 2 "Resistor_SMD:R_0805_2012Metric" H 24120 20759 30  0001 L CNN
 F 3 "" H 24050 20850 30  0000 C CNN
@@
 P 15600 4650
 F 0 "R72" V 15500 4650 50  0000 C CNN
-F 1 "100K" V 15600 4650 50  0000 C CNN
+F 1 "10k" V 15600 4650 50  0000 C CNN
 F 2 "Resistor_SMD:R_0805_2012Metric" H 15670 4559 30  0001 L CNN
 F 3 "" H 15600 4650 30  0000 C CNN
@@
 P 15600 8700
 F 0 "R162" V 15500 8700 50  0000 C CNN
-F 1 "100K" V 15600 8700 50  0000 C CNN
+F 1 "10k" V 15600 8700 50  0000 C CNN
 F 2 "Resistor_SMD:R_0805_2012Metric" H 15670 8609 30  0001 L CNN
 F 3 "" H 15600 8700 30  0000 C CNN
@@
 P 15600 12750
 F 0 "R252" V 15500 12750 50  0000 C CNN
-F 1 "100K" V 15600 12750 50  0000 C CNN
+F 1 "10k" V 15600 12750 50  0000 C CNN
 F 2 "Resistor_SMD:R_0805_2012Metric" H 15670 12659 30  0001 L CNN
 F 3 "" H 15600 12750 30  0000 C CNN
@@
 P 15600 16800
 F 0 "R342" V 15500 16800 50  0000 C CNN
-F 1 "100K" V 15600 16800 50  0000 C CNN
+F 1 "10k" V 15600 16800 50  0000 C CNN
 F 2 "Resistor_SMD:R_0805_2012Metric" H 15670 16709 30  0001 L CNN
 F 3 "" H 15600 16800 30  0000 C CNN
@@
 P 15600 20850
 F 0 "R432" V 15500 20850 50  0000 C CNN
-F 1 "100K" V 15600 20850 50  0000 C CNN
+F 1 "10k" V 15600 20850 50  0000 C CNN
 F 2 "Resistor_SMD:R_0805_2012Metric" H 15670 20759 30  0001 L CNN
 F 3 "" H 15600 20850 30  0000 C CNN
@@
 P 7300 4650
 F 0 "R71" V 7200 4650 50  0000 C CNN
-F 1 "100K" V 7300 4650 50  0000 C CNN
+F 1 "10k" V 7300 4650 50  0000 C CNN
 F 2 "Resistor_SMD:R_0805_2012Metric" H 7370 4559 30  0001 L CNN
 F 3 "" H 7300 4650 30  0000 C CNN
@@
 P 7300 8700
 F 0 "R161" V 7200 8700 50  0000 C CNN
-F 1 "100K" V 7300 8700 50  0000 C CNN
+F 1 "10k" V 7300 8700 50  0000 C CNN
 F 2 "Resistor_SMD:R_0805_2012Metric" H 7370 8609 30  0001 L CNN
 F 3 "" H 7300 8700 30  0000 C CNN
@@
 P 7300 12750
 F 0 "R251" V 7200 12750 50  0000 C CNN
-F 1 "100K" V 7300 12750 50  0000 C CNN
+F 1 "10k" V 7300 12750 50  0000 C CNN
 F 2 "Resistor_SMD:R_0805_2012Metric" H 7370 12659 30  0001 L CNN
 F 3 "" H 7300 12750 30  0000 C CNN
@@
 P 7300 16800
 F 0 "R341" V 7200 16800 50  0000 C CNN
-F 1 "100K" V 7300 16800 50  0000 C CNN
+F 1 "10k" V 7300 16800 50  0000 C CNN
 F 2 "Resistor_SMD:R_0805_2012Metric" H 7370 16709 30  0001 L CNN
 F 3 "" H 7300 16800 30  0000 C CNN
@@
 P 7300 20850
 F 0 "R431" V 7200 20850 50  0000 C CNN
-F 1 "100K" V 7300 20850 50  0000 C CNN
+F 1 "10k" V 7300 20850 50  0000 C CNN
 F 2 "Resistor_SMD:R_0805_2012Metric" H 7370 20759 30  0001 L CNN
 F 3 "" H 7300 20850 30  0000 C CNN
@@
 AR Path="/6237E8F3/6D3A924C" Ref="R?"  Part="1"
 F 0 "R468" V 43100 30950 50  0000 C CNN
-F 1 "750 Om" V 43034 30800 50  0000 C CNN
+F 1 "10k" V 43034 30800 50  0000 C CNN
 F 2 "Resistor_SMD:R_0805_2012Metric_Pad1.15x1.40mm_HandSolder" V 43080 30800 30  0001 C CNN
 F 3 "" H 43150 30800 30  0000 C CNN
@@
 AR Path="/6237E8F3/6D3A9252" Ref="R?"  Part="1"
 F 0 "R467" V 43350 30750 50  0000 C CNN
-F 1 "1k" V 43284 30600 50  0000 C CNN
-F 2 "Resistor_SMD:R_0805_2012Metric_Pad1.15x1.40mm_HandSolder" V 43330 30600 30  0001 C CNN
+F 1 "10k" V 43284 30600 50  0000 C CNN
+F 2 "Resistor_SMD:R_0805_2012Metric" V 43330 30600 30  0001 C CNN
 F 3 "" H 43400 30600 30  0000 C CNN
 	1    43400 30600
@@
 AR Path="/6237E8F3/6D3A9258" Ref="R?"  Part="1"
 F 0 "R466" V 43100 30550 50  0000 C CNN
-F 1 "1.5k" V 43034 30400 50  0000 C CNN
+F 1 "10k" V 43034 30400 50  0000 C CNN
 F 2 "Resistor_SMD:R_0805_2012Metric_Pad1.15x1.40mm_HandSolder" V 43080 30400 30  0001 C CNN
 F 3 "" H 43150 30400 30  0000 C CNN
