File: schem/LED_driver/LED_driver.kicad_pcb (KiCad board)
At the start: 2 copper layers, 922 parts, among them J1 Screw_Terminal_01x04, J10 Screw_Terminal_01x02, J11 Screw_Terminal_01x02, J12 Screw_Terminal_01x02, J13 Screw_Terminal_01x02, J14 Screw_Terminal_01x02, J15 Screw_Terminal_01x02, J16 Screw_Terminal_01x02, J17 Screw_Terminal_01x02, J18 Screw_Terminal_01x02, J19 Screw_Terminal_01x02, J2 Screw_Terminal_01x04, J20 Screw_Terminal_01x02, J21 Screw_Terminal_01x02, J22 Screw_Terminal_01x02, J23 Screw_Terminal_01x02, J24 Screw_Terminal_01x02, J25 Screw_Terminal_01x02, J26 Screw_Terminal_01x02, J27 Screw_Terminal_01x02, J28 Screw_Terminal_01x02, J29 Screw_Terminal_01x02, J3 Screw_Terminal_01x04, J30 Screw_Terminal_01x02, J31 SWD, J32 RJ45_Shielded, J33 RJ45_Shielded, J34 DEBUG, J35 Screw_Terminal_01x02, J4 Screw_Terminal_01x04, J5 Screw_Terminal_01x04, J6 Screw_Terminal_01x02, J7 Screw_Terminal_01x02, J8 Screw_Terminal_01x02, J9 Screw_Terminal_01x02, SW1 SW_DIP_x01, U1 LM3406, U10 LM3406, U11 LM3406, U12 LM3406, U13 LM3406, U14 LM3406, U15 LM3406, U16 LM3406, U17 LM3406, U18 LM3406, U19 LM3406, U2 LM3406, U20 LM3406, U21 LM3406, U22 LM3406, U23 LM3406, U24 LM3406, U25 LM3406, U26 74HC595, U27 74HC595, U28 TL431LP, U29 STM32F303VCTx, U3 LM3406, U30 MCP2551-I_SN, U31 LM1117-3.3, U32 74HC595, U33 GD25Q16C, U34 MAX3485, U35 ISO7341C, U36 LM2596S-ADJ, U37 74HC595, U4 LM3406, U5 LM3406, U6 LM3406, U7 LM3406, U8 LM3406, U9 LM3406, Y1 Crystal_Small

Commit message: Начало платы
Начертил контур платы начал расставлять разъемы.
Parts:
- moved J11 501.0 mm to (59.5, 99.2), turned to 90 degrees
- moved J6 415.2 mm to (59.5, 88.7), turned to 90 degrees
- moved J16 357.7 mm to (59.5, 109.8), turned to 90 degrees
- moved J1 322.1 mm to (59.5, 78.1), turned to 90 degrees
- moved U31 183.7 mm to (322.6, 52.1)
Other:
- board outline added: 188 x 275 mm
Changed lines of the file:
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@@
   (general
     (thickness 1.6)
-    (drawings 0)
+    (drawings 4)
     (tracks 0)
     (zones 0)
@@
     (nets 457)
   )
-  (page A4)
+  (page A3 portrait)
   (layers
     (0 F.Cu signal)
@@
     (solder_mask_min_width 0.25)
     (aux_axis_origin 0 0)
-    (visible_elements FFFFFF7F)
+    (visible_elements 7FFFFFFF)
     (pcbplotparams
       (layerselection 0x010fc_ffffffff)
@@
   )
   (module TerminalBlock:TerminalBlock_bornier-4_P5.08mm (layer F.Cu)
-    (at 377.475001 26.185001)
+    (at 59.54 78.07 90)
     (descr "simple 4-pin terminal block, pitch 5.08mm, revamped version of bornier4")
     (tags "terminal block bornier4")
-    (fp_text reference J1 (at 7.6 -4.8) (layer F.SilkS)
+    (fp_text reference J1 (at 7.6 -4.8 90) (layer F.SilkS)
       (effects (font (size 1 1) (thickness 0.15)))
     )
-    (fp_text value Screw_Terminal_01x04 (at 7.6 4.75) (layer F.Fab)
+    (fp_text value Screw_Terminal_01x04 (at 7.6 4.75 90) (layer F.Fab)
       (effects (font (size 1 1) (thickness 0.15)))
     )
-    (fp_text user %R (at 7.62 0) (layer F.Fab)
+    (fp_text user %R (at 7.62 0 90) (layer F.Fab)
       (effects (font (size 1 1) (thickness 0.15)))
     )
@@
     (fp_line (start 17.97 4) (end 17.97 -4) (layer F.CrtYd) (width 0.05))
     (fp_line (start 17.97 4) (end -2.73 4) (layer F.CrtYd) (width 0.05))
-    (pad 2 thru_hole circle (at 5.08 0) (size 3 3) (drill 1.52) (layers *.Cu *.Mask)
+    (pad 2 thru_hole circle (at 5.08 0 90) (size 3 3) (drill 1.52) (layers *.Cu *.Mask)
       (net 11 GND))
-    (pad 3 thru_hole circle (at 10.16 0) (size 3 3) (drill 1.52) (layers *.Cu *.Mask)
+    (pad 3 thru_hole circle (at 10.16 0 90) (size 3 3) (drill 1.52) (layers *.Cu *.Mask)
       (net 12 "Net-(C126-Pad1)"))
-    (pad 1 thru_hole rect (at 0 0) (size 3 3) (drill 1.52) (layers *.Cu *.Mask)
+    (pad 1 thru_hole rect (at 0 0 90) (size 3 3) (drill 1.52) (layers *.Cu *.Mask)
       (net 11 GND))
-    (pad 4 thru_hole circle (at 15.24 0) (size 3 3) (drill 1.52) (layers *.Cu *.Mask)
+    (pad 4 thru_hole circle (at 15.24 0 90) (size 3 3) (drill 1.52) (layers *.Cu *.Mask)
       (net 12 "Net-(C126-Pad1)"))
     (model ${KISYS3DMOD}/TerminalBlock.3dshapes/TerminalBlock_bornier-4_P5.08mm.wrl
@@
   )
   (module TerminalBlock:TerminalBlock_bornier-2_P5.08mm (layer F.Cu)
-    (at 473.895001 114.385001)
+    (at 59.54 88.66 90)
     (descr "simple 2-pin terminal block, pitch 5.08mm, revamped version of bornier2")
     (tags "terminal block bornier2")
-    (fp_text reference J6 (at 2.54 -5.08) (layer F.SilkS)
+    (fp_text reference J6 (at 2.54 -5.08 90) (layer F.SilkS)
       (effects (font (size 1 1) (thickness 0.15)))
     )
-    (fp_text value Screw_Terminal_01x02 (at 2.54 5.08) (layer F.Fab)
+    (fp_text value Screw_Terminal_01x02 (at 2.54 5.08 90) (layer F.Fab)
       (effects (font (size 1 1) (thickness 0.15)))
     )
-    (fp_text user %R (at 2.54 0) (layer F.Fab)
+    (fp_text user %R (at 2.54 0 90) (layer F.Fab)
       (effects (font (size 1 1) (thickness 0.15)))
     )
@@
     (fp_line (start 7.79 4) (end 7.79 -4) (layer F.CrtYd) (width 0.05))
     (fp_line (start 7.79 4) (end -2.71 4) (layer F.CrtYd) (width 0.05))
-    (pad 1 thru_hole rect (at 0 0) (size 3 3) (drill 1.52) (layers *.Cu *.Mask)
+    (pad 1 thru_hole rect (at 0 0 90) (size 3 3) (drill 1.52) (layers *.Cu *.Mask)
       (net 18 "Net-(C21-Pad1)"))
-    (pad 2 thru_hole circle (at 5.08 0) (size 3 3) (drill 1.52) (layers *.Cu *.Mask)
+    (pad 2 thru_hole circle (at 5.08 0 90) (size 3 3) (drill 1.52) (layers *.Cu *.Mask)
       (net 17 "Net-(C21-Pad2)"))
     (model ${KISYS3DMOD}/TerminalBlock.3dshapes/TerminalBlock_bornier-2_P5.08mm.wrl
@@
   )
   (module TerminalBlock:TerminalBlock_bornier-2_P5.08mm (layer F.Cu)
-    (at 555.195001 26.185001)
+    (at 59.55 99.21 90)
     (descr "simple 2-pin terminal block, pitch 5.08mm, revamped version of bornier2")
     (tags "terminal block bornier2")
-    (fp_text reference J11 (at 2.54 -5.08) (layer F.SilkS)
+    (fp_text reference J11 (at 2.54 -5.08 90) (layer F.SilkS)
       (effects (font (size 1 1) (thickness 0.15)))
     )
-    (fp_text value Screw_Terminal_01x02 (at 2.54 5.08) (layer F.Fab)
+    (fp_text value Screw_Terminal_01x02 (at 2.54 5.08 90) (layer F.Fab)
       (effects (font (size 1 1) (thickness 0.15)))
     )
@@
     (fp_line (start -2.46 -3.75) (end -2.46 3.75) (layer F.Fab) (width 0.1))
     (fp_line (start -2.41 2.55) (end 7.49 2.55) (layer F.Fab) (width 0.1))
-    (fp_text user %R (at 2.54 0) (layer F.Fab)
+    (fp_text user %R (at 2.54 0 90) (layer F.Fab)
       (effects (font (size 1 1) (thickness 0.15)))
     )
-    (pad 2 thru_hole circle (at 5.08 0) (size 3 3) (drill 1.52) (layers *.Cu *.Mask)
+    (pad 2 thru_hole circle (at 5.08 0 90) (size 3 3) (drill 1.52) (layers *.Cu *.Mask)
       (net 48 "Net-(C61-Pad2)"))
-    (pad 1 thru_hole rect (at 0 0) (size 3 3) (drill 1.52) (layers *.Cu *.Mask)
+    (pad 1 thru_hole rect (at 0 0 90) (size 3 3) (drill 1.52) (layers *.Cu *.Mask)
       (net 47 "Net-(C61-Pad1)"))
     (model ${KISYS3DMOD}/TerminalBlock.3dshapes/TerminalBlock_bornier-2_P5.08mm.wrl
@@
   )
   (module TerminalBlock:TerminalBlock_bornier-2_P5.08mm (layer F.Cu)
-    (at 412.885001 165.635001)
+    (at 59.54 109.79 90)
     (descr "simple 2-pin terminal block, pitch 5.08mm, revamped version of bornier2")
     (tags "terminal block bornier2")
-    (fp_text reference J16 (at 2.54 -5.08) (layer F.SilkS)
+    (fp_text reference J16 (at 2.54 -5.08 90) (layer F.SilkS)
       (effects (font (size 1 1) (thickness 0.15)))
     )
-    (fp_text value Screw_Terminal_01x02 (at 2.54 5.08) (layer F.Fab)
+    (fp_text value Screw_Terminal_01x02 (at 2.54 5.08 90) (layer F.Fab)
       (effects (font (size 1 1) (thickness 0.15)))
     )
@@
     (fp_line (start -2.46 -3.75) (end -2.46 3.75) (layer F.Fab) (width 0.1))
     (fp_line (start -2.41 2.55) (end 7.49 2.55) (layer F.Fab) (width 0.1))
-    (fp_text user %R (at 2.54 0) (layer F.Fab)
+    (fp_text user %R (at 2.54 0 90) (layer F.Fab)
       (effects (font (size 1 1) (thickness 0.15)))
     )
-    (pad 2 thru_hole circle (at 5.08 0) (size 3 3) (drill 1.52) (layers *.Cu *.Mask)
+    (pad 2 thru_hole circle (at 5.08 0 90) (size 3 3) (drill 1.52) (layers *.Cu *.Mask)
       (net 77 "Net-(C101-Pad2)"))
-    (pad 1 thru_hole rect (at 0 0) (size 3 3) (drill 1.52) (layers *.Cu *.Mask)
+    (pad 1 thru_hole rect (at 0 0 90) (size 3 3) (drill 1.52) (layers *.Cu *.Mask)
       (net 78 "Net-(C101-Pad1)"))
     (model ${KISYS3DMOD}/TerminalBlock.3dshapes/TerminalBlock_bornier-2_P5.08mm.wrl
@@
   )
   (module Package_TO_SOT_THT:TO-220-3_Vertical (layer F.Cu)
-    (at 505.195001 72.185001)
+    (at 322.59 52.14)
     (descr "TO-220-3, Vertical, RM 2.54mm, see https://www.vishay.com/docs/66542/to-220-1.pdf")
     (tags "TO-220-3 Vertical RM 2.54mm")
@@
     )
   )
+  (gr_line (start 243.36 326.69) (end 55.36 326.69) (layer Edge.Cuts) (width 0.05))
+  (gr_line (start 243.36 51.7) (end 243.36 326.69) (layer Edge.Cuts) (width 0.05))
+  (gr_line (start 55.38 51.69) (end 243.36 51.7) (layer Edge.Cuts) (width 0.05))
+  (gr_line (start 55.36 326.69) (end 55.38 51.69) (layer Edge.Cuts) (width 0.05))
 )

Commit message: Плата
исправил ошибку в схеме (выключение канала). Разместил детали для одного канала (ушло времен 1 час)
Parts:
- C1, C21, C31, C32, C7, C8, D11, D6, R1, R11, R17, R18, R19, R20, R21, R22, R71, R76, R81, R86: moved to B.Cu
- moved R20 558.0 mm to (70.2, 83.2), turned to 270 degrees
- moved R21 545.6 mm to (72.5, 83.2), turned to 270 degrees
- moved R23 541.8 mm to (64.8, 83.2), turned to 270 degrees
- moved R24 539.1 mm to (67.1, 83.2), turned to 270 degrees
- moved R22 532.0 mm to (74.8, 83.2), turned to 270 degrees
- moved D16 525.2 mm to (105.2, 88.0), turned to 270 degrees
- moved C7 516.9 mm to (118.6, 83.6), turned to 270 degrees
- moved R17 502.8 mm to (63.2, 83.2), turned to 270 degrees
- moved R81 499.4 mm to (105.3, 88.9), turned to 180 degrees
- moved C21 499.3 mm to (79.5, 88.2), turned to 180 degrees
- moved R19 491.2 mm to (67.8, 83.2), turned to 270 degrees
- moved D1 486.1 mm to (99.7, 85.1), turned to 270 degrees
- moved R16 482.9 mm to (113.0, 85.9)
- moved D6 475.4 mm to (92.4, 85.1), turned to 270 degrees
- moved C8 471.4 mm to (112.2, 80.3), turned to 90 degrees
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Connections:
- D101 pad 5: (no net) -> Net-(D101-Pad5)
- D11 pad 3: Net-(C126-Pad1) -> Net-(D11-Pad3)
- D12 pad 3: Net-(C10-Pad1) -> Net-(D12-Pad3)
- D13 pad 3: Net-(C12-Pad1) -> Net-(D13-Pad3)
- D14 pad 3: Net-(C135-Pad1) -> Net-(D14-Pad3)
- D15 pad 3: Net-(C100-Pad1) -> Net-(D15-Pad3)
- D31 pad 3: Net-(C126-Pad1) -> Net-(D31-Pad3)
- D32 pad 3: Net-(C10-Pad1) -> Net-(D32-Pad3)
- D33 pad 3: Net-(C12-Pad1) -> Net-(D33-Pad3)
- D34 pad 3: Net-(C135-Pad1) -> Net-(D34-Pad3)
- D35 pad 3: Net-(C100-Pad1) -> Net-(D35-Pad3)
- D51 pad 3: Net-(C126-Pad1) -> Net-(D51-Pad3)
- D52 pad 3: Net-(C10-Pad1) -> Net-(D52-Pad3)
- D53 pad 3: Net-(C12-Pad1) -> Net-(D53-Pad3)
- D54 pad 3: Net-(C135-Pad1) -> Net-(D54-Pad3)
- D55 pad 3: Net-(C100-Pad1) -> Net-(D55-Pad3)
- D71 pad 3: Net-(C126-Pad1) -> Net-(D71-Pad3)
- D72 pad 3: Net-(C10-Pad1) -> Net-(D72-Pad3)
- D73 pad 3: Net-(C12-Pad1) -> Net-(D73-Pad3)
- D74 pad 3: Net-(C135-Pad1) -> Net-(D74-Pad3)
- D75 pad 3: Net-(C100-Pad1) -> Net-(D75-Pad3)
- D91 pad 3: Net-(C126-Pad1) -> Net-(D91-Pad3)
- D92 pad 3: Net-(C10-Pad1) -> Net-(D92-Pad3)
- D93 pad 3: Net-(C12-Pad1) -> Net-(D93-Pad3)
- D94 pad 3: Net-(C135-Pad1) -> Net-(D94-Pad3)
- D95 pad 3: Net-(C100-Pad1) -> Net-(D95-Pad3)
- J31 pad 5: (no net) -> Net-(J31-Pad5)
- J32 pad 5: (no net) -> Net-(J32-Pad5)
- J32 pad 6: (no net) -> Net-(J32-Pad6)
- J33 pad 5: (no net) -> Net-(J33-Pad5)
- J33 pad 6: (no net) -> Net-(J33-Pad6)
- R10 pad 1: Net-(R10-Pad1) -> Net-(D15-Pad3)
- R100 pad 1: Net-(R100-Pad1) -> Net-(D35-Pad3)
- R186 pad 1: Net-(R186-Pad1) -> Net-(D51-Pad3)
- R187 pad 1: Net-(R187-Pad1) -> Net-(D52-Pad3)
- R188 pad 1: Net-(R188-Pad1) -> Net-(D53-Pad3)
- R189 pad 1: Net-(R189-Pad1) -> Net-(D54-Pad3)
- R190 pad 1: Net-(R190-Pad1) -> Net-(D55-Pad3)
- R276 pad 1: Net-(R276-Pad1) -> Net-(D71-Pad3)
- R277 pad 1: Net-(R277-Pad1) -> Net-(D72-Pad3)
- R278 pad 1: Net-(R278-Pad1) -> Net-(D73-Pad3)
- R279 pad 1: Net-(R279-Pad1) -> Net-(D74-Pad3)
- R280 pad 1: Net-(R280-Pad1) -> Net-(D75-Pad3)
- R366 pad 1: Net-(R366-Pad1) -> Net-(D91-Pad3)
- R367 pad 1: Net-(R367-Pad1) -> Net-(D92-Pad3)
- R368 pad 1: Net-(R368-Pad1) -> Net-(D93-Pad3)
- R369 pad 1: Net-(R369-Pad1) -> Net-(D94-Pad3)
- R370 pad 1: Net-(R370-Pad1) -> Net-(D95-Pad3)
- R6 pad 1: Net-(R6-Pad1) -> Net-(D11-Pad3)
- R7 pad 1: Net-(R7-Pad1) -> Net-(D12-Pad3)
- R8 pad 1: Net-(R8-Pad1) -> Net-(D13-Pad3)
- R9 pad 1: Net-(R9-Pad1) -> Net-(D14-Pad3)
- R96 pad 1: Net-(R96-Pad1) -> Net-(D31-Pad3)
- R97 pad 1: Net-(R97-Pad1) -> Net-(D32-Pad3)
- R98 pad 1: Net-(R98-Pad1) -> Net-(D33-Pad3)
- R99 pad 1: Net-(R99-Pad1) -> Net-(D34-Pad3)
- U1 pad 10: Net-(R6-Pad1) -> Net-(D11-Pad3)
- U1 pad 4: (no net) -> Net-(U1-Pad4)
- U10 pad 10: Net-(R100-Pad1) -> Net-(D35-Pad3)
- U10 pad 4: (no net) -> Net-(U10-Pad4)
- U11 pad 10: Net-(R186-Pad1) -> Net-(D51-Pad3)
- U11 pad 4: (no net) -> Net-(U11-Pad4)
- U12 pad 10: Net-(R187-Pad1) -> Net-(D52-Pad3)
- U12 pad 4: (no net) -> Net-(U12-Pad4)
- U13 pad 10: Net-(R188-Pad1) -> Net-(D53-Pad3)
- U13 pad 4: (no net) -> Net-(U13-Pad4)
- U14 pad 10: Net-(R189-Pad1) -> Net-(D54-Pad3)
- U14 pad 4: (no net) -> Net-(U14-Pad4)
- U15 pad 10: Net-(R190-Pad1) -> Net-(D55-Pad3)
- U15 pad 4: (no net) -> Net-(U15-Pad4)
- U16 pad 10: Net-(R276-Pad1) -> Net-(D71-Pad3)
- U16 pad 4: (no net) -> Net-(U16-Pad4)
- U17 pad 10: Net-(R277-Pad1) -> Net-(D72-Pad3)
- U17 pad 4: (no net) -> Net-(U17-Pad4)
- U18 pad 10: Net-(R278-Pad1) -> Net-(D73-Pad3)
- U18 pad 4: (no net) -> Net-(U18-Pad4)
- U19 pad 10: Net-(R279-Pad1) -> Net-(D74-Pad3)
- U19 pad 4: (no net) -> Net-(U19-Pad4)
- U2 pad 10: Net-(R7-Pad1) -> Net-(D12-Pad3)
- U2 pad 4: (no net) -> Net-(U2-Pad4)
- U20 pad 10: Net-(R280-Pad1) -> Net-(D75-Pad3)
- U20 pad 4: (no net) -> Net-(U20-Pad4)
- U21 pad 10: Net-(R366-Pad1) -> Net-(D91-Pad3)
- U21 pad 4: (no net) -> Net-(U21-Pad4)
- U22 pad 10: Net-(R367-Pad1) -> Net-(D92-Pad3)
- U22 pad 4: (no net) -> Net-(U22-Pad4)
- U23 pad 10: Net-(R368-Pad1) -> Net-(D93-Pad3)
- U23 pad 4: (no net) -> Net-(U23-Pad4)
- U24 pad 10: Net-(R369-Pad1) -> Net-(D94-Pad3)
- U24 pad 4: (no net) -> Net-(U24-Pad4)
- U25 pad 10: Net-(R370-Pad1) -> Net-(D95-Pad3)
- U25 pad 4: (no net) -> Net-(U25-Pad4)
- U3 pad 10: Net-(R8-Pad1) -> Net-(D13-Pad3)
- U3 pad 4: (no net) -> Net-(U3-Pad4)
- U30 pad 5: (no net) -> Net-(U30-Pad5)
- U35 pad 14: (no net) -> Net-(U35-Pad14)
- U35 pad 3: (no net) -> Net-(U35-Pad3)
- U37 pad 4: (no net) -> Net-(U37-Pad4)
- U37 pad 5: (no net) -> Net-(U37-Pad5)
- U37 pad 6: (no net) -> Net-(U37-Pad6)
- U37 pad 7: (no net) -> Net-(U37-Pad7)
- U37 pad 9: (no net) -> Net-(U37-Pad9)
- U4 pad 10: Net-(R9-Pad1) -> Net-(D14-Pad3)
- U4 pad 4: (no net) -> Net-(U4-Pad4)
- U5 pad 10: Net-(R10-Pad1) -> Net-(D15-Pad3)
- U5 pad 4: (no net) -> Net-(U5-Pad4)
- U6 pad 10: Net-(R96-Pad1) -> Net-(D31-Pad3)
- U6 pad 4: (no net) -> Net-(U6-Pad4)
- U7 pad 10: Net-(R97-Pad1) -> Net-(D32-Pad3)
- U7 pad 4: (no net) -> Net-(U7-Pad4)
- U8 pad 10: Net-(R98-Pad1) -> Net-(D33-Pad3)
- U8 pad 4: (no net) -> Net-(U8-Pad4)
- U9 pad 10: Net-(R99-Pad1) -> Net-(D34-Pad3)
- U9 pad 4: (no net) -> Net-(U9-Pad4)

Commit message: 1
Parts:
- moved C6 1.83 mm to (120.8, 82.6)
- moved C7 1.74 mm to (118.9, 85.3)
- moved C8 1.65 mm to (112.1, 82.0)
Changed lines of the file:
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@@
   )
   (module Capacitor_THT:CP_Radial_D10.0mm_P5.00mm (layer F.Cu)
-    (at 120.78 80.76 270)
+    (at 120.83 82.59 270)
     (descr "CP, Radial series, Radial, pin pitch=5.00mm, , diameter=10mm, Electrolytic Capacitor")
     (tags "CP Radial series Radial pin pitch 5.00mm  diameter 10mm Electrolytic Capacitor")
@@
   )
   (module Capacitor_SMD:C_0805_2012Metric (layer B.Cu)
-    (at 118.57 83.62 270)
+    (at 118.9 85.33 270)
     (descr "Capacitor SMD 0805 (2012 Metric), square (rectangular) end terminal, IPC_7351 nominal, (Body size source: https://docs.google.com/spreadsheets/d/1BsfQQcO9C6DZCsRaXUlFlo91Tg2WpOkGARC1WS5S8t0/edit?usp=sharing), generated with kicad-footprint-generator")
     (tags capacitor)
@@
   )
   (module Capacitor_SMD:C_0805_2012Metric (layer B.Cu)
-    (at 112.17 80.33 90)
+    (at 112.08 81.98 90)
     (descr "Capacitor SMD 0805 (2012 Metric), square (rectangular) end terminal, IPC_7351 nominal, (Body size source: https://docs.google.com/spreadsheets/d/1BsfQQcO9C6DZCsRaXUlFlo91Tg2WpOkGARC1WS5S8t0/edit?usp=sharing), generated with kicad-footprint-generator")
     (tags capacitor)
@@
     (descr "CP, Radial series, Radial, pin pitch=5.00mm, , diameter=10mm, Electrolytic Capacitor")
     (tags "CP Radial series Radial pin pitch 5.00mm  diameter 10mm Electrolytic Capacitor")
-    (fp_text reference C22 (at 2.5 -6.25 180) (layer F.SilkS)
+    (fp_text reference C22 (at -1.59 -5 180) (layer F.SilkS)
       (effects (font (size 1 1) (thickness 0.15)))
     )
@@
     (tags "Diode SMC (DO-214AB)")
     (attr smd)
-    (fp_text reference D1 (at 0 -4.1 270) (layer F.SilkS)
+    (fp_text reference D1 (at 6.106 0.01 270) (layer F.SilkS)
       (effects (font (size 1 1) (thickness 0.15)))
     )
@@
     (tags "Choke SMD")
     (attr smd)
-    (fp_text reference L1 (at 6.47 -4.77) (layer F.SilkS)
+    (fp_text reference L1 (at 5.196 -6.35) (layer F.SilkS)
       (effects (font (size 1 1) (thickness 0.15)))
     )
@@
     (tags "SSOP 0.65 exposed pad")
     (attr smd)
-    (fp_text reference U1 (at 0 -3.55) (layer F.SilkS)
+    (fp_text reference U1 (at 2.02 3.726) (layer F.SilkS)
       (effects (font (size 1 1) (thickness 0.15)))
     )

Commit message: Плата
Parts:
- removed the C21 at (79.5, 88.2)
- removed the C31 at (109.5, 86.9)
- removed the D11 at (114.2, 86.6)
- removed the R76 at (100.5, 87.6)
- added C1: 0.1mkF, Capacitor_SMD:C_0805_2012Metric, B.Cu at (99.9, 148.9)
- added C1: 0.1mkF, Capacitor_SMD:C_0805_2012Metric, B.Cu at (99.9, 131.9)
- added C101: 0.1mkF, Capacitor_SMD:C_0805_2012Metric, F.Cu at (73.5, 121.6)
- added C102: 470mkF, Capacitor_THT:CP_Radial_D10.0mm_P5.00mm, F.Cu at (82.4, 119.0)
- added C111: 0.1mkF, Capacitor_SMD:C_0805_2012Metric, B.Cu at (110.7, 121.3)
- added C112: 1mkF, Capacitor_SMD:C_0805_2012Metric, B.Cu at (110.7, 123.3)
- added C21: 0.1mkF, Capacitor_SMD:C_0805_2012Metric, F.Cu at (73.5, 155.6)
- added C21: 0.1mkF, Capacitor_SMD:C_0805_2012Metric, F.Cu at (73.5, 138.6)
- added C21: 0.1mkF, Capacitor_SMD:C_0805_2012Metric, F.Cu at (73.5, 87.6)
- added C22: 470mkF, Capacitor_THT:CP_Radial_D10.0mm_P5.00mm, F.Cu at (82.4, 153.0)
- added C22: 470mkF, Capacitor_THT:CP_Radial_D10.0mm_P5.00mm, F.Cu at (82.4, 136.0)
- added C31: 0.1mkF, Capacitor_SMD:C_0805_2012Metric, B.Cu at (110.7, 155.3)
- added C31: 0.1mkF, Capacitor_SMD:C_0805_2012Metric, B.Cu at (110.7, 138.3)
- added C31: 0.1mkF, Capacitor_SMD:C_0805_2012Metric, B.Cu at (110.7, 87.3)
- added C32: 1mkF, Capacitor_SMD:C_0805_2012Metric, B.Cu at (110.7, 157.3)
- added C32: 1mkF, Capacitor_SMD:C_0805_2012Metric, B.Cu at (110.7, 140.3)
- added C41: 0.1mkF, Capacitor_SMD:C_0805_2012Metric, B.Cu at (99.9, 97.9)
- added C46: 470mkF, Capacitor_THT:CP_Radial_D10.0mm_P5.00mm, F.Cu at (120.8, 99.6)
- added C47: 0.1mkF, Capacitor_SMD:C_0805_2012Metric, B.Cu at (118.9, 102.3)
- added C48: 0.1mkF, Capacitor_SMD:C_0805_2012Metric, B.Cu at (112.9, 98.2)
- added C6: 470mkF, Capacitor_THT:CP_Radial_D10.0mm_P5.00mm, F.Cu at (120.8, 150.6)
- added C6: 470mkF, Capacitor_THT:CP_Radial_D10.0mm_P5.00mm, F.Cu at (120.8, 133.6)
- added C61: 0.1mkF, Capacitor_SMD:C_0805_2012Metric, F.Cu at (73.5, 104.6)
- added C62: 470mkF, Capacitor_THT:CP_Radial_D10.0mm_P5.00mm, F.Cu at (82.4, 102.0)
- added C7: 0.1mkF, Capacitor_SMD:C_0805_2012Metric, B.Cu at (118.9, 153.3)
- added C7: 0.1mkF, Capacitor_SMD:C_0805_2012Metric, B.Cu at (118.9, 136.3)
- added C71: 0.1mkF, Capacitor_SMD:C_0805_2012Metric, B.Cu at (110.7, 104.3)
- added C72: 1mkF, Capacitor_SMD:C_0805_2012Metric, B.Cu at (110.7, 106.3)
- added C8: 0.1mkF, Capacitor_SMD:C_0805_2012Metric, B.Cu at (112.9, 149.2)
- added C8: 0.1mkF, Capacitor_SMD:C_0805_2012Metric, B.Cu at (112.9, 132.2)
- added C81: 0.1mkF, Capacitor_SMD:C_0805_2012Metric, B.Cu at (99.9, 114.9)
- added C86: 470mkF, Capacitor_THT:CP_Radial_D10.0mm_P5.00mm, F.Cu at (120.8, 116.6)
- added C87: 0.1mkF, Capacitor_SMD:C_0805_2012Metric, B.Cu at (118.9, 119.3)
- added C88: 0.1mkF, Capacitor_SMD:C_0805_2012Metric, B.Cu at (112.9, 115.2)
- added D1: D_Schottky, Diode_SMD:D_SMC, F.Cu at (99.8, 152.8)
- added D1: D_Schottky, Diode_SMD:D_SMC, F.Cu at (99.8, 135.8)
- added D11: Si2300, Package_TO_SOT_SMD:SOT-23, B.Cu at (115.3, 154.6)
- added D11: Si2300, Package_TO_SOT_SMD:SOT-23, B.Cu at (115.3, 137.6)
- added D11: Si2300, Package_TO_SOT_SMD:SOT-23, B.Cu at (115.3, 86.6)
- added D16: lmc7101, Package_TO_SOT_SMD:SOT-23-5, B.Cu at (82.2, 149.5)
- added D16: lmc7101, Package_TO_SOT_SMD:SOT-23-5, B.Cu at (82.2, 132.5)
- added D21: D_Schottky, Diode_SMD:D_SMC, F.Cu at (99.8, 101.8)
- added D26: D_Schottky, Diode_SMD:D_SMC, B.Cu at (92.4, 102.1)
- added D31: Si2300, Package_TO_SOT_SMD:SOT-23, B.Cu at (115.3, 103.6)
- added D36: lmc7101, Package_TO_SOT_SMD:SOT-23-5, B.Cu at (82.2, 98.5)
- added D41: D_Schottky, Diode_SMD:D_SMC, F.Cu at (99.8, 118.8)
- added D46: D_Schottky, Diode_SMD:D_SMC, B.Cu at (92.4, 119.1)
- added D51: Si2300, Package_TO_SOT_SMD:SOT-23, B.Cu at (115.3, 120.6)
- added D56: lmc7101, Package_TO_SOT_SMD:SOT-23-5, B.Cu at (82.2, 115.5)
- added D6: D_Schottky, Diode_SMD:D_SMC, B.Cu at (92.4, 153.1)
- added D6: D_Schottky, Diode_SMD:D_SMC, B.Cu at (92.4, 136.1)
- added J11: Screw_Terminal_01x02, TerminalBlock:TerminalBlock_bornier-2_P5.08mm, F.Cu at (59.5, 105.7)
- added J16: Screw_Terminal_01x02, TerminalBlock:TerminalBlock_bornier-2_P5.08mm, F.Cu at (59.5, 122.7)
- added J6: Screw_Terminal_01x02, TerminalBlock:TerminalBlock_bornier-2_P5.08mm, F.Cu at (59.5, 156.7)
- added J6: Screw_Terminal_01x02, TerminalBlock:TerminalBlock_bornier-2_P5.08mm, F.Cu at (59.5, 139.7)
- added L1: 22mkH, Inductor_SMD:L_10.4x10.4_H4.8, F.Cu at (90.8, 153.9)
- added L1: 22mkH, Inductor_SMD:L_10.4x10.4_H4.8, F.Cu at (90.8, 136.9)
- added L11: 22mkH, Inductor_SMD:L_10.4x10.4_H4.8, F.Cu at (90.8, 119.9)
- added L6: 22mkH, Inductor_SMD:L_10.4x10.4_H4.8, F.Cu at (90.8, 102.9)
- added R1: 1K, Resistor_SMD:R_0805_2012Metric, B.Cu at (100.5, 151.7)
- added R1: 1K, Resistor_SMD:R_0805_2012Metric, B.Cu at (100.5, 134.7)
- added R101: 1K, Resistor_SMD:R_0805_2012Metric, B.Cu at (100.5, 102.7)
- added R106: 100, Resistor_SMD:R_0805_2012Metric, F.Cu at (113.0, 102.9)
- added R107: 1R, Resistor_SMD:R_1206_3216Metric, B.Cu at (63.2, 100.2)
- added R108: 1R, Resistor_SMD:R_1206_3216Metric, B.Cu at (65.5, 100.2)
- added R109: 1R, Resistor_SMD:R_1206_3216Metric, B.Cu at (67.8, 100.2)
- added R11: 1K, Resistor_SMD:R_0805_2012Metric, B.Cu at (100.5, 153.7)
- added R11: 1K, Resistor_SMD:R_0805_2012Metric, B.Cu at (100.5, 136.7)
- added R110: 1R, Resistor_SMD:R_1206_3216Metric, B.Cu at (70.2, 100.2)
- added R111: 1R, Resistor_SMD:R_1206_3216Metric, B.Cu at (72.5, 100.2)
- added R112: 1R, Resistor_SMD:R_1206_3216Metric, B.Cu at (74.8, 100.2)
- added R113: 1R, Resistor_SMD:R_1206_3216Metric, F.Cu at (71.7, 100.2)
- added R114: 1R, Resistor_SMD:R_1206_3216Metric, F.Cu at (69.4, 100.2)
- added R115: 1R, Resistor_SMD:R_1206_3216Metric, F.Cu at (67.1, 100.2)
- added R116: 1R, Resistor_SMD:R_1206_3216Metric, F.Cu at (64.8, 100.2)
- added R16: 100, Resistor_SMD:R_0805_2012Metric, F.Cu at (113.0, 153.9)
- added R16: 100, Resistor_SMD:R_0805_2012Metric, F.Cu at (113.0, 136.9)
- added R161: 100K, Resistor_SMD:R_0805_2012Metric, B.Cu at (115.3, 106.4)
- added R166: 1K, Resistor_SMD:R_0805_2012Metric, B.Cu at (78.3, 99.5)
- added R17: 1R, Resistor_SMD:R_1206_3216Metric, B.Cu at (63.2, 151.2)
- added R17: 1R, Resistor_SMD:R_1206_3216Metric, B.Cu at (63.2, 134.2)
- added R171: 1K, Resistor_SMD:R_0805_2012Metric, B.Cu at (78.3, 97.5)
- added R176: 10K, Resistor_SMD:R_0805_2012Metric, B.Cu at (85.1, 98.5)
- added R18: 1R, Resistor_SMD:R_1206_3216Metric, B.Cu at (65.5, 151.2)
- added R18: 1R, Resistor_SMD:R_1206_3216Metric, B.Cu at (65.5, 134.2)
- added R181: 1K, Resistor_SMD:R_0805_2012Metric, B.Cu at (100.5, 117.7)
- added R186: 100K, Resistor_SMD:R_0805_2012Metric, B.Cu at (116.3, 117.0)
- added R19: 1R, Resistor_SMD:R_1206_3216Metric, B.Cu at (67.8, 151.2)
- added R19: 1R, Resistor_SMD:R_1206_3216Metric, B.Cu at (67.8, 134.2)
- added R191: 1K, Resistor_SMD:R_0805_2012Metric, B.Cu at (100.5, 119.7)
- added R196: 100, Resistor_SMD:R_0805_2012Metric, F.Cu at (113.0, 119.9)
- added R197: 1R, Resistor_SMD:R_1206_3216Metric, B.Cu at (63.2, 117.2)
- added R198: 1R, Resistor_SMD:R_1206_3216Metric, B.Cu at (65.5, 117.2)
- added R199: 1R, Resistor_SMD:R_1206_3216Metric, B.Cu at (67.8, 117.2)
- added R20: 1R, Resistor_SMD:R_1206_3216Metric, B.Cu at (70.2, 151.2)
- added R20: 1R, Resistor_SMD:R_1206_3216Metric, B.Cu at (70.2, 134.2)
- added R200: 1R, Resistor_SMD:R_1206_3216Metric, B.Cu at (70.2, 117.2)
- added R201: 1R, Resistor_SMD:R_1206_3216Metric, B.Cu at (72.5, 117.2)
- added R202: 1R, Resistor_SMD:R_1206_3216Metric, B.Cu at (74.8, 117.2)
- added R203: 1R, Resistor_SMD:R_1206_3216Metric, F.Cu at (64.8, 117.2)
- added R204: 1R, Resistor_SMD:R_1206_3216Metric, F.Cu at (67.1, 117.2)
- added R205: 1R, Resistor_SMD:R_1206_3216Metric, F.Cu at (69.4, 117.2)
- added R206: 1R, Resistor_SMD:R_1206_3216Metric, F.Cu at (71.7, 117.2)
- added R21: 1R, Resistor_SMD:R_1206_3216Metric, B.Cu at (72.5, 151.2)
- added R21: 1R, Resistor_SMD:R_1206_3216Metric, B.Cu at (72.5, 134.2)
- added R22: 1R, Resistor_SMD:R_1206_3216Metric, B.Cu at (74.8, 151.2)
- added R22: 1R, Resistor_SMD:R_1206_3216Metric, B.Cu at (74.8, 134.2)
- added R23: 1R, Resistor_SMD:R_1206_3216Metric, F.Cu at (64.8, 151.2)
- added R23: 1R, Resistor_SMD:R_1206_3216Metric, F.Cu at (64.8, 134.2)
- added R24: 1R, Resistor_SMD:R_1206_3216Metric, F.Cu at (67.1, 151.2)
- added R24: 1R, Resistor_SMD:R_1206_3216Metric, F.Cu at (67.1, 134.2)
- added R25: 1R, Resistor_SMD:R_1206_3216Metric, F.Cu at (69.4, 151.2)
- added R25: 1R, Resistor_SMD:R_1206_3216Metric, F.Cu at (69.4, 134.2)
- added R251: 100K, Resistor_SMD:R_0805_2012Metric, B.Cu at (115.3, 123.4)
- added R256: 1K, Resistor_SMD:R_0805_2012Metric, B.Cu at (78.3, 116.5)
- added R26: 1R, Resistor_SMD:R_1206_3216Metric, F.Cu at (71.7, 151.2)
- added R26: 1R, Resistor_SMD:R_1206_3216Metric, F.Cu at (71.7, 134.2)
- added R261: 1K, Resistor_SMD:R_0805_2012Metric, B.Cu at (78.3, 114.5)
- added R266: 10K, Resistor_SMD:R_0805_2012Metric, B.Cu at (85.1, 115.5)
- added R6: 100K, Resistor_SMD:R_0805_2012Metric, B.Cu at (116.3, 151.0)
- added R6: 100K, Resistor_SMD:R_0805_2012Metric, B.Cu at (116.3, 134.0)
- added R6: 100K, Resistor_SMD:R_0805_2012Metric, B.Cu at (116.3, 100.0)
- added R71: 100K, Resistor_SMD:R_0805_2012Metric, B.Cu at (115.3, 157.4)
- added R71: 100K, Resistor_SMD:R_0805_2012Metric, B.Cu at (115.3, 140.4)
- added R76: 1K, Resistor_SMD:R_0805_2012Metric, B.Cu at (78.3, 150.5)
- added R76: 1K, Resistor_SMD:R_0805_2012Metric, B.Cu at (78.3, 133.5)
- added R76: 1K, Resistor_SMD:R_0805_2012Metric, B.Cu at (78.3, 82.5)
- added R81: 1K, Resistor_SMD:R_0805_2012Metric, B.Cu at (78.3, 148.5)
- added R81: 1K, Resistor_SMD:R_0805_2012Metric, B.Cu at (78.3, 131.5)
- added R86: 10K, Resistor_SMD:R_0805_2012Metric, B.Cu at (85.1, 149.5)
- added R86: 10K, Resistor_SMD:R_0805_2012Metric, B.Cu at (85.1, 132.5)
- added R91: 1K, Resistor_SMD:R_0805_2012Metric, B.Cu at (100.5, 100.7)
- added U1: LM3406, Package_SO:TSSOP-14-1EP_4.4x5mm_P0.65mm, F.Cu at (107.2, 151.1)
- added U1: LM3406, Package_SO:TSSOP-14-1EP_4.4x5mm_P0.65mm, F.Cu at (107.2, 134.1)
- added U11: LM3406, Package_SO:TSSOP-14-1EP_4.4x5mm_P0.65mm, F.Cu at (107.2, 117.1)
- added U6: LM3406, Package_SO:TSSOP-14-1EP_4.4x5mm_P0.65mm, F.Cu at (107.2, 100.1)
- D16, R6: moved to B.Cu
- moved J11 250.0 mm to (307.8, 128.7)
- moved J16 250.0 mm to (307.8, 139.3)
- moved J21 250.0 mm to (307.8, 149.9)
- moved J26 250.0 mm to (307.8, 160.5)
- moved R81 28.2 mm to (78.3, 80.5), turned to 0 degrees
- moved D16 24.0 mm to (82.2, 81.5), turned to 90 degrees
- moved R86 20.9 mm to (85.1, 81.5), turned to 270 degrees
- moved R6 2.73 mm to (116.3, 83.0), turned to 90 degrees
- moved C1 1.52 mm to (99.9, 80.9)
- moved C32 1.25 mm to (110.7, 89.3)
- moved C8 1.18 mm to (112.9, 81.2), turned to 180 degrees
- moved R71 1.07 mm to (115.3, 89.4)
- moved C22 0.97 mm to (82.4, 85.0)
- moved D1 0.31 mm to (99.8, 84.8)
Routing:
- net Net-(C21-Pad2): track 0.00 -> 495.3 mm, vias 0 -> 30
- net Net-(C21-Pad1): track 0.00 -> 340.8 mm
- net Net-(C126-Pad1): track 0.00 -> 270.4 mm, vias 0 -> 5
- net GND: track 0.00 -> 270.1 mm, vias 0 -> 35
- net Net-(C1-Pad1): track 0.00 -> 70.5 mm, vias 0 -> 5
- net Net-(C32-Pad1): track 0.00 -> 49.7 mm, vias 0 -> 5
- net Net-(D11-Pad3): track 0.00 -> 47.3 mm, vias 0 -> 5
- net Net-(D16-Pad4): track 0.00 -> 41.7 mm
- net Net-(C1-Pad2): track 0.00 -> 33.0 mm, vias 0 -> 5
- net Net-(C31-Pad1): track 0.00 -> 21.9 mm, vias 0 -> 5
- net Net-(R11-Pad2): track 0.00 -> 18.1 mm, vias 0 -> 5
- net Net-(R1-Pad2): track 0.00 -> 14.2 mm, vias 0 -> 5
- net Net-(R16-Pad1): track 0.00 -> 13.0 mm
- net /Isens_CH1: track 0.00 -> 10.4 mm
- net Net-(D16-Pad3): track 0.00 -> 9.87 mm
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- added copper zone on F.Cu, net Net-(C1-Pad1)
- added copper zone on B.Cu, net Net-(C21-Pad2)
- added copper zone on F.Cu, net Net-(C21-Pad2)
