File: schem/LED_driver/LED_driver.kicad_pcb (KiCad board)
At the start: 2 copper layers, 188 x 275 mm, 1054 parts, among them J1 Screw_Terminal_01x04, J10 Screw_Terminal_01x02, J11 Screw_Terminal_01x02, J12 Screw_Terminal_01x02, J13 Screw_Terminal_01x02, J14 Screw_Terminal_01x02, J15 Screw_Terminal_01x02, J16 Screw_Terminal_01x02, J17 Screw_Terminal_01x02, J18 Screw_Terminal_01x02, J19 Screw_Terminal_01x02, J2 Screw_Terminal_01x04, J20 Screw_Terminal_01x02, J21 Screw_Terminal_01x02, J22 Screw_Terminal_01x02, J23 Screw_Terminal_01x02, J24 Screw_Terminal_01x02, J25 Screw_Terminal_01x02, J26 Screw_Terminal_01x02, J27 Screw_Terminal_01x02, J28 Screw_Terminal_01x02, J29 Screw_Terminal_01x02, J3 Screw_Terminal_01x04, J30 Screw_Terminal_01x02, J31 SWD, J32 RJ45_Shielded, J33 RJ45_Shielded, J34 DEBUG, J35 Screw_Terminal_01x02, J4 Screw_Terminal_01x04, J5 Screw_Terminal_01x04, J6 Screw_Terminal_01x02, J7 Screw_Terminal_01x02, J8 Screw_Terminal_01x02, J9 Screw_Terminal_01x02, SW1 SW_DIP_x01, U1 LM3406, U10 LM3406, U11 LM3406, U12 LM3406, U13 LM3406, U14 LM3406, U15 LM3406, U16 LM3406, U17 LM3406, U18 LM3406, U19 LM3406, U2 LM3406, U20 LM3406, U21 LM3406, U22 LM3406, U23 LM3406, U24 LM3406, U25 LM3406, U26 74HC595, U27 74HC595, U28 TL431LP, U29 STM32F303VCTx, U3 LM3406, U30 MCP2551-I_SN, U31 LM1117-3.3, U32 74HC595, U33 GD25Q16C, U34 MAX3485, U35 ISO7341C, U36 LM2596S-ADJ, U37 74HC595, U4 LM3406, U5 LM3406, U6 LM3406, U7 LM3406, U8 LM3406, U9 LM3406, Y1 Crystal_Small

Commit message: Плата
Закончил разводку 5 каналов
Parts:
- removed the L1 at (90.8, 153.9)
- removed the R71 at (115.3, 140.4)
- added L21: 22mkH, Inductor_SMD:L_10.4x10.4_H4.8, F.Cu at (90.8, 153.9)
- added R341: 100K, Resistor_SMD:R_0805_2012Metric, B.Cu at (115.3, 140.4)
- renumbered C1 to C121, C6 to C126, C7 to C127, C8 to C128, C21 to C141, C22 to C142, C31 to C151, C32 to C152, C1 to C161, C6 to C166, C7 to C167, C8 to C168, C21 to C181, C22 to C182, C31 to C191, C32 to C192, D1 to D61, D6 to D66, D11 to D71, D16 to D76, D1 to D81, D6 to D86, D11 to D91, D16 to D96, J6 to J21, J6 to J26, L1 to L16, R1 to R271, R6 to R276, R11 to R281, R16 to R286, R17 to R287, R18 to R288, R19 to R289, R20 to R290, R21 to R291, R22 to R292, R23 to R293, R24 to R294, R25 to R295, R26 to R296, R76 to R346, R81 to R351, R86 to R356, R1 to R361, R6 to R366, R11 to R371, R16 to R376, R17 to R377, R18 to R378, R19 to R379, R20 to R380, R21 to R381, R22 to R382, R23 to R383, R24 to R384, R25 to R385, R26 to R386, R71 to R431, R76 to R436, R81 to R441, R86 to R446, U1 to U16, U1 to U21
